File: poly_kb_mainboard/SSD1306_TO_SPI.sch (KiCad schematic (older format))
At the start: 10 parts, among them J14 Conn_01x16, J15 Conn_01x01_Female, J19 Conn_01x01_Male

Commit message: PolyKB almost final dual-board version
Parts:
- removed C19: 1uF, Capacitor_SMD:C_0805_2012Metric, symbol Device:C_Small
- removed C21: 2.2uF, Capacitor_SMD:C_0805_2012Metric, symbol Device:C_Small
- removed J15: Conn_01x01_Female, Connector_PinHeader_1.00mm:PinHeader_1x01_P1.00mm_Vertical, symbol Connector:Conn_01x01_Female
- removed J19: Conn_01x01_Male, Connector_PinHeader_1.00mm:PinHeader_1x01_P1.00mm_Vertical, symbol Connector:Conn_01x01_Male
- added C144: 1uF, Capacitor_SMD:C_0402_1005Metric, symbol Device:C_Small
- added C146: 2.2uF, Capacitor_SMD:C_0603_1608Metric, symbol Device:C_Small
- C18: footprint Capacitor_SMD:C_0805_2012Metric -> Capacitor_SMD:C_0402_1005Metric; LCSC C28323 -> C52923
- C20: footprint Capacitor_SMD:C_0805_2012Metric -> Capacitor_SMD:C_0603_1608Metric; LCSC C49217 -> C23630
- C22: footprint Capacitor_SMD:C_0805_2012Metric -> Capacitor_SMD:C_0402_1005Metric; LCSC C1779 -> C23733
- C23: footprint Capacitor_SMD:C_0805_2012Metric -> Capacitor_SMD:C_0402_1005Metric; LCSC C49678 -> C1525
- LED_1: LCSC C114583 -> C527089
Connections:
- net CS: now also J14.10 (Pin_10)
- net GND: now also C146.2
- net at J14.15 (Pin_15): now also C146.1
- net at J14.6 (Pin_6): now also C144.1
- net at J14.7 (Pin_7): now also C144.2
Other:
- moved on the sheet: J141
