File: poly_kb_mainboard/poly_kb.sch (KiCad schematic (older format))
At the start: 53 parts, among them J1 SWD, J2 USB_C_Receptacle_USB2.0, J3 Left, J4 Right, J5 USART2, J6 I2C1, J7 Bottom, J8 Conn_01x02, SW1 Boot0, SW2 Boot1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

Commit message: Added Python scripts to translate BOM and CPL
Parts:
- J1: LCSC (none) -> C225520
Changed lines of the file:
@@
 F 2 "poly_kb:SIDE-SWD" H 7850 -8200 50  0001 C CNN
 F 3 "~" H 7850 -8200 50  0001 C CNN
+F 4 "C225520" H 7850 -8200 50  0001 C CNN "LCSC"
 	1    7850 -8200
 	1    0    0    -1

Commit message: PolyKB almost final dual-board version
Parts:
- removed C1, C2, C3, C4: 1u, Capacitor_SMD:C_0402_1005Metric, symbol Device:C_Small
- removed C10, C11, C12, C13, C7, C8, C9: 100n, Capacitor_SMD:C_0402_1005Metric, symbol Device:C_Small
- removed C14, C15: 2u2, Capacitor_SMD:C_0603_1608Metric, symbol Device:C_Small
- removed C16, C17: 12p, Capacitor_SMD:C_0402_1005Metric, symbol Device:C_Small
- removed C5: 10n, Capacitor_SMD:C_0402_1005Metric, symbol Device:C_Small
- removed C6: 4u7, Capacitor_SMD:C_0603_1608Metric, symbol Device:C_Small
- removed D1: Reset, LED_SMD:LED_0603_1608Metric, symbol Device:LED_Small
- removed D2: Status, LED_SMD:LED_0603_1608Metric, symbol Device:LED_Small
- removed D3: Power, LED_SMD:LED_0603_1608Metric, symbol Device:LED_Small
- removed F1: 2A, Fuse:Fuse_1206_3216Metric, symbol Device:Polyfuse_Small
- removed FB1, FB2: 600 @ 600 MHz, Inductor_SMD:L_0805_2012Metric, symbol Device:Ferrite_Bead_Small
- removed J1: SWD, poly_kb:SIDE-SWD, symbol Connector_Generic:Conn_02x05_Odd_Even
- removed J2: USB_C_Receptacle_USB2.0, Connector_USB:USB_C_Receptacle_HRO_TYPE-C-31-M-12, symbol Connector:USB_C_Receptacle_USB2.0
- removed J3: Left, Connector_PinHeader_2.54mm:PinHeader_2x06_P2.54mm_Vertical, symbol Connector_Generic:Conn_02x06_Top_Bottom
- removed J4: Right, Connector_PinHeader_2.54mm:PinHeader_1x12_P2.54mm_Vertical, symbol Connector_Generic:Conn_01x12
- removed J5: USART2, Connector_PinHeader_2.54mm:PinHeader_2x04_P2.54mm_Vertical, symbol Connector_Generic:Conn_02x04_Odd_Even
- removed J6: I2C1, Connector_PinHeader_2.54mm:PinHeader_1x04_P2.54mm_Vertical, symbol Connector_Generic:Conn_01x04
- removed J7: Bottom, Connector_PinHeader_2.54mm:PinHeader_2x20_P2.54mm_Vertical, symbol Connector_Generic:Conn_02x20_Counter_Clockwise
- removed J8: Conn_01x02, Connector_PinHeader_2.54mm:PinHeader_1x02_P2.54mm_Vertical, symbol Connector_Generic:Conn_01x02
- removed R1, R3: 100k, Resistor_SMD:R_0402_1005Metric, symbol Device:R_Small
- removed R10, R11: 5k1, Resistor_SMD:R_0402_1005Metric, symbol Device:R_Small
- removed R12, R6, R7: 1k5, Resistor_SMD:R_0402_1005Metric, symbol Device:R_Small
- removed R13: 47, Resistor_SMD:R_0402_1005Metric, symbol Device:R_Small
- removed R14, R15, R2: 10k, Resistor_SMD:R_0402_1005Metric, symbol Device:R_Small
- removed R4, R5, R8, R9: 22, Resistor_SMD:R_0402_1005Metric, symbol Device:R_Small
- removed SW1: Boot0, Button_Switch_SMD:SW_SPST_B3U-3000P-B, symbol Switch:SW_SPST
- removed SW2: Boot1, Button_Switch_SMD:SW_SPST_B3U-3000P-B, symbol Switch:SW_SPST
- removed SW3: Reset, Button_Switch_SMD:SW_SPST_B3U-3000P-B, symbol Switch:SW_SPST
- removed U1: XC6206P332MR, Package_TO_SOT_SMD:SOT-23, symbol Regulator_Linear:XC6206PxxxMR
- removed U2: STM32F407VETx, Package_QFP:LQFP-100_14x14mm_P0.5mm, symbol MCU_ST_STM32F4:STM32F407VETx
- removed U3: W25N01GVZEIG, poly_kb:W25N01GVZEIG, symbol poly_kb:W25N01GVZEIG-SchmillipKiCADLibrary
- removed Y1: 16MHz, Crystal:Crystal_SMD_3225-4Pin_3.2x2.5mm, symbol Device:Crystal_GND24_Small
Connections:
- no-connect marks 5 -> 0
Other:
- note removed: "128MByte SPI Flash"
- note removed: "3.3V@5A Power Supply"
- note removed: "Blue\n"
- note removed: "Boot Switches"
- note removed: "Debug Interface SWD"
- note removed: "External High Speed XTAL"
- note removed: "Green"
- note removed: "I2C 1 Interface\nStatus Display"
- note removed: "Mainboard Interface"
- note removed: "Power Supply via USB C"
- note removed: "Red"
- note removed: "Reset Switch"
- note removed: "Status LEDs"
- note removed: "VDD/GND Pairs"
- note removed: "VDDA Decoupling"
