File: poly_kb_atom/SSD1306_TO_SPI.sch (KiCad schematic (older format))
At the start: 10 parts, among them J14 Conn_01x16, SW1 SW_Push

Commit message: Fixed wrong connection in between pin 16 an VCC in PolyAtom2; Added ConectorL
Connections:
- net 3V3: no longer C20.1, J14.16 (Pin_16)
- new net: C20.1, J14.16 (Pin_16)
Changed lines of the file:
@@
 encoding utf-8
 Sheet 3 3
-Title ""
-Date ""
-Rev ""
-Comp ""
+Title "Display Adapter, LED & Switch"
+Date "2022-01-24"
+Rev "2.1"
+Comp "thpoll"
 Comment1 ""
 Comment2 ""
@@
 	4950 4750 4950 4900
 Wire Wire Line
-	4250 4550 4950 4550
-Connection ~ 4950 4550
-Wire Wire Line
 	4950 4550 5200 4550
 Text HLabel 4650 4450 0    50   Input ~ 0
@@
 Text HLabel 4950 4900 3    50   Input ~ 0
 GND
-Text HLabel 4250 4550 0    50   Input ~ 0
-3V3
 Text HLabel 3800 3850 0    50   Input ~ 0
 3V3
