File: poly_kb_atom/poly_kb_1.5U.kicad_pcb (KiCad board)
At the start: 2 copper layers, 28.6 x 19 mm, 18 parts, among them J1 Conn_01x16, J2 North, J3 WestFront, J4 EastFront, J5 WestBack, J6 EastBack, J7 South, J8 North2, J9 South2, SW1 SW_Push

Commit message: Added new revisions for all pcbs expect 1.25U; cleaned up gerber dirs
Parts:
- added R1: 1M, Resistor_SMD:R_0402_1005Metric, B.Cu at (95.6, 60.4)
- added kibuzzard-61EFA8F1: G***, kibuzzard-61EFA8F1, F.Cu at (112.7, 69.7)
- added kibuzzard-61EFAA6D: G***, kibuzzard-61EFAA6D, F.Cu at (113.0, 63.7)
- added kibuzzard-61EFABBF: G***, kibuzzard-61EFABBF, F.Cu at (112.8, 67.7)
- added kibuzzard-61EFACF9: G***, kibuzzard-61EFACF9, F.Cu at (112.2, 59.7)
- added kibuzzard-61EFBE21: G***, kibuzzard-61EFBE21, F.Cu at (90.3, 65.7)
- added kibuzzard-61EFBE2C: G***, kibuzzard-61EFBE2C, F.Cu at (90.7, 67.7)
- added kibuzzard-61EFBE3D: G***, kibuzzard-61EFBE3D, F.Cu at (90.8, 69.7)
- added kibuzzard-61EFBE87: G***, kibuzzard-61EFBE87, F.Cu at (91.3, 59.7)
- added kibuzzard-61EFD7F9: G***, kibuzzard-61EFD7F9, F.Cu at (113.1, 65.7)
- added kibuzzard-61EFD863: G***, kibuzzard-61EFD863, F.Cu at (112.4, 57.7)
- added kibuzzard-61EFD879: G***, kibuzzard-61EFD879, F.Cu at (91.1, 57.7)
- added kibuzzard-61EFD908: G***, kibuzzard-61EFD908, F.Cu at (89.9, 71.7)
- added kibuzzard-61EFD908: G***, kibuzzard-61EFD908, F.Cu at (113.6, 71.7)
- added kibuzzard-61EFD947: G***, kibuzzard-61EFD947, F.Cu at (113.6, 55.7)
- added kibuzzard-61EFD947: G***, kibuzzard-61EFD947, F.Cu at (89.9, 55.7)
- added kibuzzard-61EFDAA0: G***, kibuzzard-61EFDAA0, F.Cu at (90.2, 61.7)
- added kibuzzard-61EFDAC6: G***, kibuzzard-61EFDAC6, F.Cu at (113.6, 61.7)
- added kibuzzard-61EFDAEE: G***, kibuzzard-61EFDAEE, F.Cu at (90.5, 63.7)
- added kibuzzard-6209778F: G***, kibuzzard-6209778F, F.Cu at (99.5, 72.0)
- D1: footprint Diode_SMD:D_SOD-323 -> poly_kb:D_SOD-323Ext
- LED1: value WS2812B-Mini -> LED
- moved C4 177.1 mm to (104.3, 61.8)
- moved D1 177.0 mm to (98.4, 67.0)
- moved C3 177.0 mm to (95.1, 56.9)
- moved C6 177.0 mm to (100.5, 61.4)
- moved J3 177.0 mm to (88.5, 63.7)
- moved J4 177.0 mm to (115.0, 63.7)
- moved J5 177.0 mm to (88.5, 63.7)
- moved J6 177.0 mm to (115.0, 63.7)
- moved J7 177.0 mm to (95.8, 72.4)
- moved J8 177.0 mm to (95.8, 54.9)
- moved SW1 177.0 mm to (104.3, 59.9)
- moved J1 177.0 mm to (101.7, 58.0)
- moved J2 177.0 mm to (107.7, 54.9)
- moved J9 177.0 mm to (107.7, 72.4)
- moved LED1 177.0 mm to (101.7, 56.1)
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Connections:
- C1 pad 1: /Keyboard/sheet605ED2EB/3V3 -> Net-(C1-Pad1)
- J1 pad 16: /Keyboard/sheet605ED2EB/3V3 -> Net-(C1-Pad1)
- J1 pad 2: (no net) -> unconnected-(J1-Pad2)
- J3 pad 4: /Keyboard/sheet605ED2EB/LED_DOUT -> /Keyboard/sheet605ED2EB/LED_DIN
- LED1 pad 2: /Keyboard/sheet605ED2EB/LED_DOUT -> /Keyboard/sheet605ED2EB/LED_DIN
Routing:
- net /Keyboard/sheet605ED2EB/LED_DIN: track 17.3 -> 33.1 mm, vias 2 -> 4
- net /Keyboard/sheet605ED2EB/LED_DOUT: track 15.3 -> 0.00 mm, vias 2 -> 0
- net Net-(C1-Pad1): track 0.00 -> 6.05 mm
- net /Keyboard/sheet605ED2EB/CS: track 47.5 -> 50.5 mm
- net /Keyboard/sheet605ED2EB/GND: track 45.8 -> 48.4 mm, vias 5 -> 20
- net /Keyboard/sheet605ED2EB/3V3: track 35.8 -> 33.4 mm
- net /Keyboard/sheet605ED2EB/SCLK: track 45.3 -> 46.8 mm
- net /Keyboard/sheet605ED2EB/D-C: track 45.4 -> 44.0 mm
- net /Keyboard/sheet605ED2EB/SDIN: track 40.5 -> 41.8 mm
- net /Keyboard/sheet605ED2EB/RESET: track 33.3 -> 34.5 mm
- net CS2: track 28.9 -> 29.9 mm
- net CS8: track 27.9 -> 28.9 mm
- net Net-(C5-Pad2): track 2.46 -> 1.78 mm
- net Net-(D1-Pad2): track 6.52 -> 5.85 mm
- added copper zone on B.Cu, net /Keyboard/sheet605ED2EB/GND
- added copper zone on F.Cu, net /Keyboard/sheet605ED2EB/GND
Other:
- outline, holes or cut-outs redrawn
- net class Default removed
- board text added: ".1"
- board text added: "16"
- board text added: "C3"
- board text added: "D"
- board text added: "E"
- board text added: "JLCJLCJLCJLC"
- board text added: "L"
- board text removed: "1.5U"
- board text removed: "3V3"
- board text removed: "CLK"
- board text removed: "D\C"
- board text removed: "GND"
- board text removed: "PCBPUYPCBPUY"
- board text removed: "RST"
- board text removed: "SI"
- board text removed: "VBAT"
- board text removed: "i"
- board text removed: "o"
- board text removed: "pick one"
- board text removed: "r"

Commit message: Added optional C7 and fix LED silkscreens
Parts:
- added C7: 100nF, Capacitor_SMD:C_0603_1608Metric, F.Cu at (97.7, 56.0)
- LED1: value LED -> WS2812B-Mini
Changed lines of the file:
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@@
       (effects (font (size 0.6 0.6) (thickness 0.15)))
     )
-    (fp_text value "LED" (at 0 0 180) (layer "F.Fab")
+    (fp_text value "WS2812B-Mini" (at 0 0 180) (layer "F.Fab")
       (effects (font (size 0.6 0.6) (thickness 0.15)))
     )
-    (fp_text user "+" (at -2.5 -1) (layer "F.SilkS")
-      (effects (font (size 1 1) (thickness 0.15)))
-    )
-    (fp_text user "o" (at -2.5 0.8) (layer "F.SilkS")
-      (effects (font (size 1 1) (thickness 0.15)))
-    )
-    (fp_text user "i" (at 2.5 -0.8) (layer "F.SilkS")
-      (effects (font (size 1 1) (thickness 0.15)))
-    )
-    (fp_text user "-" (at 2.5 0.8) (layer "F.SilkS")
-      (effects (font (size 1 1) (thickness 0.15)))
-    )
+    (fp_text user "+" (at -2.5 -1) (layer "F.SilkS") hide
+      (effects (font (size 1 1) (thickness 0.15)))
+    )
+    (fp_text user "o" (at -2.5 0.8) (layer "F.SilkS") hide
+      (effects (font (size 1 1) (thickness 0.15)))
+    )
+    (fp_text user "i" (at 2.5 -0.8) (layer "F.SilkS") hide
+      (effects (font (size 1 1) (thickness 0.15)))
+    )
+    (fp_text user "-" (at 2.5 0.8) (layer "F.SilkS") hide
+      (effects (font (size 1 1) (thickness 0.15)))
+    )
+    (fp_line (start 0.94 1.74) (end -1.74 1.74) (layer "F.SilkS") (width 0.12))
     (fp_line (start -1.74 -1.74) (end -1.74 -1.5) (layer "F.SilkS") (width 0.12))
     (fp_line (start 0.94 1.74) (end 1.7 1.74) (layer "F.SilkS") (width 0.12))
-    (fp_line (start 0.94 1.74) (end -1.74 1.74) (layer "F.SilkS") (width 0.12))
     (fp_line (start 1.74 -1.74) (end 1.74 -1.5) (layer "F.SilkS") (width 0.12))
+    (fp_line (start -1.74 -1.74) (end 1.74 -1.74) (layer "F.SilkS") (width 0.12))
     (fp_line (start -1.74 1.74) (end -1.74 1.5) (layer "F.SilkS") (width 0.12))
-    (fp_line (start -1.74 -1.74) (end 1.74 -1.74) (layer "F.SilkS") (width 0.12))
+    (fp_poly (pts
+        (xy 2.9 1.45)
+        (xy 2.392 1.45)
+        (xy 2.9 0.942)
+      ) (layer "F.SilkS") (width 0.12) (fill solid))
     (fp_line (start 1.74 -1.74) (end -1.74 -1.74) (layer "F.CrtYd") (width 0.05))
     (fp_line (start -1.74 1.74) (end -1.74 -1.74) (layer "F.CrtYd") (width 0.05))
+    (fp_line (start 1.74 1.74) (end 1.74 -1.74) (layer "F.CrtYd") (width 0.05))
     (fp_line (start -1.74 1.74) (end 1.74 1.74) (layer "F.CrtYd") (width 0.05))
-    (fp_line (start 1.74 1.74) (end 1.74 -1.74) (layer "F.CrtYd") (width 0.05))
-    (pad "1" smd rect locked (at -1.365 -0.89 90) (size 0.8 0.95) (layers "F.Cu" "F.Paste" "F.Mask")
+    (pad "1" smd rect (at -1.465 -0.89 90) (size 0.9 1.15) (layers "F.Cu" "F.Paste" "F.Mask")
       (net 15 "/Keyboard/sheet605ED2EB/5V") (pinfunction "VDD") (pintype "power_in"))
-    (pad "2" smd rect locked (at -1.365 0.89 90) (size 0.8 0.95) (layers "F.Cu" "F.Paste" "F.Mask")
+    (pad "2" smd rect (at -1.465 0.89 90) (size 0.9 1.15) (layers "F.Cu" "F.Paste" "F.Mask")
       (net 14 "/Keyboard/sheet605ED2EB/LED_DIN") (pinfunction "DOUT") (pintype "output"))
-    (pad "3" smd rect locked (at 1.365 0.89 90) (size 0.8 0.95) (layers "F.Cu" "F.Paste" "F.Mask")
+    (pad "3" smd rect (at 1.465 0.89 90) (size 0.9 1.15) (layers "F.Cu" "F.Paste" "F.Mask")
       (net 1 "/Keyboard/sheet605ED2EB/GND") (pinfunction "VSS") (pintype "power_in"))
-    (pad "4" smd rect locked (at 1.365 -0.89 90) (size 0.8 0.95) (layers "F.Cu" "F.Paste" "F.Mask")
+    (pad "4" smd rect (at 1.465 -0.89 90) (size 0.9 1.15) (layers "F.Cu" "F.Paste" "F.Mask")
       (net 14 "/Keyboard/sheet605ED2EB/LED_DIN") (pinfunction "DIN") (pintype "input"))
     (model "${KIPRJMOD}/WS2812B-Mini/WS2812B-Mini.step"
@@
       ) (layer "F.SilkS") (width 0) (fill solid))
   )
+  (footprint "Capacitor_SMD:C_0603_1608Metric" (layer "F.Cu")
+    (at 97.7265 56.0448 -90)
+    (descr "Capacitor SMD 0603 (1608 Metric), square (rectangular) end terminal, IPC_7351 nominal, (Body size source: IPC-SM-782 page 76, https://www.pcb-3d.com/wordpress/wp-content/uploads/ipc-sm-782a_amendment_1_and_2.pdf), generated with kicad-footprint-generator")
+    (tags "capacitor")
+    (property "LCSC" "C19666")
+    (property "Sheetfile" "SSD1306_TO_SPI.kicad_sch")
+    (property "Sheetname" "sheet605ED2EB")
+    (attr smd)
+    (fp_text reference "C7" (at 0 -1.43 90) (layer "F.SilkS")
+      (effects (font (size 0.8 0.8) (thickness 0.15)))
+    )
+    (fp_text value "100nF" (at 0 1.43 90) (layer "F.Fab")
+      (effects (font (size 1 1) (thickness 0.15)))
+    )
+    (fp_text user "${REFERENCE}" (at 0 0 90) (layer "F.Fab")
+      (effects (font (size 0.4 0.4) (thickness 0.06)))
+    )
+    (fp_line (start -0.14058 0.51) (end 0.14058 0.51) (layer "F.SilkS") (width 0.12))
+    (fp_line (start -0.14058 -0.51) (end 0.14058 -0.51) (layer "F.SilkS") (width 0.12))
+    (fp_line (start 1.48 0.73) (end -1.48 0.73) (layer "F.CrtYd") (width 0.05))
+    (fp_line (start -1.48 0.73) (end -1.48 -0.73) (layer "F.CrtYd") (width 0.05))
+    (fp_line (start -1.48 -0.73) (end 1.48 -0.73) (layer "F.CrtYd") (width 0.05))
+    (fp_line (start 1.48 -0.73) (end 1.48 0.73) (layer "F.CrtYd") (width 0.05))
+    (fp_line (start 0.8 -0.4) (end 0.8 0.4) (layer "F.Fab") (width 0.1))
+    (fp_line (start -0.8 -0.4) (end 0.8 -0.4) (layer "F.Fab") (width 0.1))
+    (fp_line (start 0.8 0.4) (end -0.8 0.4) (layer "F.Fab") (width 0.1))
+    (fp_line (start -0.8 0.4) (end -0.8 -0.4) (layer "F.Fab") (width 0.1))
+    (pad "1" smd roundrect (at -0.775 0 270) (size 0.9 0.95) (layers "F.Cu" "F.Paste" "F.Mask") (roundrect_rratio 0.25)
+      (net 15 "/Keyboard/sheet605ED2EB/5V") (pintype "passive"))
+    (pad "2" smd roundrect (at 0.775 0 270) (size 0.9 0.95) (layers "F.Cu" "F.Paste" "F.Mask") (roundrect_rratio 0.25)
+      (net 1 "/Keyboard/sheet605ED2EB/GND") (pintype "passive"))
+    (model "${KICAD6_3DMODEL_DIR}/Capacitor_SMD.3dshapes/C_0603_1608Metric.wrl"
+      (offset (xyz 0 0 0))
+      (scale (xyz 1 1 1))
+      (rotate (xyz 0 0 0))
+    )
+  )
   (footprint "kibuzzard-61EFBE87" (layer "F.Cu")
