File: poly_kb_atom/poly_kb_1.75U.kicad_pcb (KiCad board)
At the start: 2 copper layers, 33.3 x 19 mm, 18 parts, among them J1 Conn_01x16, J2 North, J3 WestFront, J4 EastFront, J5 WestBack, J6 EastBack, J7 South, J8 North2, J9 South2, SW1 SW_Push

Commit message: Added new revisions for all pcbs expect 1.25U; cleaned up gerber dirs
Parts:
- added J10: North2, poly_kb:TestPoin_1.5x1.5mm_Drill0.7mm, F.Cu at (88.6, 54.9)
- added J2: North, poly_kb:TestPoin_1.5x1.5mm_Drill0.7mm, F.Cu at (114.8, 54.9)
- added J7: South, poly_kb:TestPoin_1.5x1.5mm_Drill0.7mm, F.Cu at (88.6, 72.4)
- added J9: South2, poly_kb:TestPoin_1.5x1.5mm_Drill0.7mm, F.Cu at (114.8, 72.4)
- added R1: 1M, Resistor_SMD:R_0402_1005Metric, B.Cu at (95.6, 60.4)
- added kibuzzard-61EFA8F1: G***, kibuzzard-61EFA8F1, F.Cu at (115.1, 69.7)
- added kibuzzard-61EFAA6D: G***, kibuzzard-61EFAA6D, F.Cu at (115.4, 63.7)
- added kibuzzard-61EFABBF: G***, kibuzzard-61EFABBF, F.Cu at (115.2, 67.7)
- added kibuzzard-61EFACF9: G***, kibuzzard-61EFACF9, F.Cu at (114.6, 59.7)
- added kibuzzard-61EFBE21: G***, kibuzzard-61EFBE21, F.Cu at (87.9, 65.7)
- added kibuzzard-61EFBE2C: G***, kibuzzard-61EFBE2C, F.Cu at (88.3, 67.7)
- added kibuzzard-61EFBE3D: G***, kibuzzard-61EFBE3D, F.Cu at (88.4, 69.7)
- added kibuzzard-61EFBE87: G***, kibuzzard-61EFBE87, F.Cu at (88.9, 59.7)
- added kibuzzard-61EFD7F9: G***, kibuzzard-61EFD7F9, F.Cu at (115.5, 65.7)
- added kibuzzard-61EFD863: G***, kibuzzard-61EFD863, F.Cu at (114.8, 57.7)
- added kibuzzard-61EFD879: G***, kibuzzard-61EFD879, F.Cu at (88.7, 57.7)
- added kibuzzard-61EFD908: G***, kibuzzard-61EFD908, F.Cu at (87.5, 71.7)
- added kibuzzard-61EFD908: G***, kibuzzard-61EFD908, F.Cu at (116.0, 71.7)
- added kibuzzard-61EFD947: G***, kibuzzard-61EFD947, F.Cu at (116.0, 55.7)
- added kibuzzard-61EFD947: G***, kibuzzard-61EFD947, F.Cu at (87.5, 55.7)
- added kibuzzard-61EFDAA0: G***, kibuzzard-61EFDAA0, F.Cu at (87.8, 61.7)
- added kibuzzard-61EFDAC6: G***, kibuzzard-61EFDAC6, F.Cu at (115.9, 61.7)
- added kibuzzard-61EFDAEE: G***, kibuzzard-61EFDAEE, F.Cu at (88.1, 63.7)
- added kibuzzard-62061ACF: G***, kibuzzard-62061ACF, F.Cu at (99.6, 72.0)
- D1: footprint Diode_SMD:D_SOD-323 -> poly_kb:D_SOD-323Ext
- moved C4 154.6 mm to (104.3, 61.8)
- moved D1 154.4 mm to (98.4, 67.0)
- moved C6 154.4 mm to (100.5, 61.4)
- moved J2 154.4 mm to (107.7, 54.9)
- moved J4 154.4 mm to (117.4, 63.7)
- moved J6 154.4 mm to (117.4, 63.7)
- moved J7 154.4 mm to (95.8, 72.4)
- moved J8 154.4 mm to (95.8, 54.9)
- moved J9 154.4 mm to (107.7, 72.4)
- moved SW1 154.4 mm to (104.3, 59.9)
- moved C3 154.4 mm to (95.1, 56.9)
- moved J1 154.4 mm to (101.7, 58.0)
- moved J3 154.4 mm to (86.1, 63.7)
- moved J5 154.4 mm to (86.1, 63.7)
- moved LED1 154.4 mm to (101.7, 56.1)
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Connections:
- C1 pad 1: /Keyboard/sheet605ED2EB/3V3 -> Net-(C1-Pad1)
- J1 pad 16: /Keyboard/sheet605ED2EB/3V3 -> Net-(C1-Pad1)
- J1 pad 2: (no net) -> unconnected-(J1-Pad2)
- J3 pad 4: /Keyboard/sheet605ED2EB/LED_DOUT -> /Keyboard/sheet605ED2EB/LED_DIN
- LED1 pad 2: /Keyboard/sheet605ED2EB/LED_DOUT -> /Keyboard/sheet605ED2EB/LED_DIN
Routing:
- net /Keyboard/sheet605ED2EB/KeyCol: track 54.6 -> 86.9 mm
- net /Keyboard/sheet605ED2EB/LED_DIN: track 19.7 -> 39.2 mm, vias 2 -> 4
- net /Keyboard/sheet605ED2EB/LED_DOUT: track 17.7 -> 0.00 mm, vias 2 -> 0
- net Net-(C1-Pad1): track 0.00 -> 6.05 mm
- net /Keyboard/sheet605ED2EB/GND: track 50.6 -> 53.7 mm, vias 5 -> 37
- net /Keyboard/sheet605ED2EB/SCLK: track 50.1 -> 52.3 mm
- net /Keyboard/sheet605ED2EB/5V: track 32.6 -> 33.9 mm
- net CS5: track 35.9 -> 34.7 mm
- net /Keyboard/sheet605ED2EB/SDIN: track 45.5 -> 46.5 mm
- net /Keyboard/sheet605ED2EB/CS: track 57.0 -> 57.9 mm
- net CS1: track 34.2 -> 33.4 mm
- net Net-(C5-Pad2): track 2.46 -> 1.78 mm
- net Net-(D1-Pad2): track 6.52 -> 5.85 mm
- net CS2: track 34.1 -> 34.7 mm
- net CS4: track 35.4 -> 36.0 mm
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- added copper zone on B.Cu, net /Keyboard/sheet605ED2EB/GND
- added copper zone on F.Cu, net /Keyboard/sheet605ED2EB/GND
Other:
- outline, holes or cut-outs redrawn
- net class Default removed
- board text added: ".1"
- board text added: "16"
- board text added: "C3"
- board text added: "D"
- board text added: "E"
- board text added: "JLCJLCJLCJLC"
- board text added: "L"
- board text removed: "1.75U"
- board text removed: "3V3"
- board text removed: "CLK"
- board text removed: "D\C"
- board text removed: "GND"
- board text removed: "PCBPUYPCBPUY"
- board text removed: "RST"
- board text removed: "SI"
- board text removed: "VBAT"
- board text removed: "i"
- board text removed: "o"
- board text removed: "pick one"
- board text removed: "r"

Commit message: Added optional C7 and fix LED silkscreens
Parts:
- added C7: 100nF, Capacitor_SMD:C_0603_1608Metric, F.Cu at (97.7, 56.1)
Changed lines of the file:
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@@
       ) (layer "F.SilkS") (width 0) (fill solid))
+  )
+  (footprint "poly_kb:TestPoin_1.5x1.5mm_Drill0.7mm" (layer "F.Cu")
+    (at 88.61425 54.9148)
+    (descr "THT rectangular pad as test Point, square 1.5mm side length, hole diameter 0.7mm")
+    (tags "test point THT pad rectangle square")
+    (property "Sheetfile" "keyboard.kicad_sch")
+    (property "Sheetname" "Keyboard")
+    (attr exclude_from_pos_files)
+    (fp_text reference "J10" (at -1.143 0) (layer "F.SilkS") hide
+      (effects (font (size 0.8 0.8) (thickness 0.153)))
+    )
+    (fp_text value "North2" (at 0 -3.4417) (layer "F.Fab")
+      (effects (font (size 1 1) (thickness 0.15)))
+    )
+    (fp_text user "${REFERENCE}" (at 0 -1.65) (layer "F.Fab") hide
+      (effects (font (size 1 1) (thickness 0.15)))
+    )
+    (pad "1" thru_hole rect locked (at 0 0) (size 1.5 1.5) (drill 0.7) (layers *.Cu *.Mask)
+      (net 18 "/Keyboard/sheet605ED2EB/KeyCol") (pinfunction "Pin_1") (pintype "passive"))
   )
   (footprint "kibuzzard-61EFA8F1" (layer "F.Cu")
@@
         (xy -0.25236 -0.585258)
       ) (layer "F.SilkS") (width 0) (fill solid))
+  )
+  (footprint "Capacitor_SMD:C_0603_1608Metric" (layer "F.Cu")
+    (at 97.7265 56.0578 -90)
+    (descr "Capacitor SMD 0603 (1608 Metric), square (rectangular) end terminal, IPC_7351 nominal, (Body size source: IPC-SM-782 page 76, https://www.pcb-3d.com/wordpress/wp-content/uploads/ipc-sm-782a_amendment_1_and_2.pdf), generated with kicad-footprint-generator")
+    (tags "capacitor")
+    (property "LCSC" "C19666")
+    (property "Sheetfile" "SSD1306_TO_SPI.kicad_sch")
+    (property "Sheetname" "sheet605ED2EB")
+    (attr smd)
+    (fp_text reference "C7" (at 0 -1.43 90) (layer "F.SilkS")
+      (effects (font (size 0.8 0.8) (thickness 0.15)))
+    )
+    (fp_text value "100nF" (at 0 1.43 90) (layer "F.Fab")
+      (effects (font (size 1 1) (thickness 0.15)))
+    )
+    (fp_text user "${REFERENCE}" (at 0 0 90) (layer "F.Fab")
+      (effects (font (size 0.4 0.4) (thickness 0.06)))
+    )
+    (fp_line (start -0.14058 0.51) (end 0.14058 0.51) (layer "F.SilkS") (width 0.12))
+    (fp_line (start -0.14058 -0.51) (end 0.14058 -0.51) (layer "F.SilkS") (width 0.12))
+    (fp_line (start 1.48 -0.73) (end 1.48 0.73) (layer "F.CrtYd") (width 0.05))
+    (fp_line (start -1.48 -0.73) (end 1.48 -0.73) (layer "F.CrtYd") (width 0.05))
+    (fp_line (start 1.48 0.73) (end -1.48 0.73) (layer "F.CrtYd") (width 0.05))
+    (fp_line (start -1.48 0.73) (end -1.48 -0.73) (layer "F.CrtYd") (width 0.05))
+    (fp_line (start -0.8 -0.4) (end 0.8 -0.4) (layer "F.Fab") (width 0.1))
+    (fp_line (start 0.8 0.4) (end -0.8 0.4) (layer "F.Fab") (width 0.1))
+    (fp_line (start -0.8 0.4) (end -0.8 -0.4) (layer "F.Fab") (width 0.1))
+    (fp_line (start 0.8 -0.4) (end 0.8 0.4) (layer "F.Fab") (width 0.1))
+    (pad "1" smd roundrect (at -0.775 0 270) (size 0.9 0.95) (layers "F.Cu" "F.Paste" "F.Mask") (roundrect_rratio 0.25)
+      (net 15 "/Keyboard/sheet605ED2EB/5V") (pintype "passive"))
+    (pad "2" smd roundrect (at 0.775 0 270) (size 0.9 0.95) (layers "F.Cu" "F.Paste" "F.Mask") (roundrect_rratio 0.25)
+      (net 1 "/Keyboard/sheet605ED2EB/GND") (pintype "passive"))
+    (model "${KICAD6_3DMODEL_DIR}/Capacitor_SMD.3dshapes/C_0603_1608Metric.wrl"
+      (offset (xyz 0 0 0))
+      (scale (xyz 1 1 1))
+      (rotate (xyz 0 0 0))
+    )
   )
   (footprint "kibuzzard-61EFD863" (layer "F.Cu")
@@
       ) (layer "F.SilkS") (width 0) (fill solid))
   )
-  (footprint "poly_kb:TestPoin_1.5x1.5mm_Drill0.7mm" (layer "F.Cu")
-    (at 88.61425 54.9148)
-    (descr "THT rectangular pad as test Point, square 1.5mm side length, hole diameter 0.7mm")
-    (tags "test point THT pad rectangle square")
-    (property "Sheetfile" "keyboard.kicad_sch")
-    (property "Sheetname" "Keyboard")
-    (attr exclude_from_pos_files)
-    (fp_text reference "J10" (at -1.143 0) (layer "F.SilkS") hide
-      (effects (font (size 0.8 0.8) (thickness 0.153)))
-    )
-    (fp_text value "North2" (at 0 -3.4417) (layer "F.Fab")
-      (effects (font (size 1 1) (thickness 0.15)))
-    )
-    (fp_text user "${REFERENCE}" (at 0 -1.65) (layer "F.Fab") hide
-      (effects (font (size 1 1) (thickness 0.15)))
-    )
-    (pad "1" thru_hole rect locked (at 0 0) (size 1.5 1.5) (drill 0.7) (layers *.Cu *.Mask)
-      (net 18 "/Keyboard/sheet605ED2EB/KeyCol") (pinfunction "Pin_1") (pintype "passive"))
-  )
   (footprint "kibuzzard-61EFABBF" (layer "F.Cu")
