File: poly_kb_atom/poly_kb_molecule_1.5x4.kicad_pcb (KiCad board)
At the start: 2 copper layers, 28.6 x 76.2 mm, 140 parts, among them J1 Conn_01x16, J2 North, J3 WestFront, J4 EastFront, J5 WestBack, J6 EastBack, J7 South, J8 North2, J9 South2, SW1 SW_Push

Commit message: Added optional C7 and fix LED silkscreens
Parts:
- added C7: 100nF, Capacitor_SMD:C_0603_1608Metric, F.Cu at (59.6, 56.1)
- added C7: 100nF, Capacitor_SMD:C_0603_1608Metric, F.Cu at (59.6, 94.2)
- added C7: 100nF, Capacitor_SMD:C_0603_1608Metric, F.Cu at (59.6, 37.0)
- added C7: 100nF, Capacitor_SMD:C_0603_1608Metric, F.Cu at (59.6, 75.1)
- LED1 (x4): value LED -> WS2812B-Mini
