File: poly_kb_atom/poly_kb_molecule_1x4.kicad_pcb (KiCad board)
At the start: 2 copper layers, 19.1 x 76.2 mm, 140 parts, among them J1 Conn_01x16, J2 North, J3 WestFront, J4 EastFront, J5 WestBack, J6 EastBack, J7 South, J8 North2, J9 South2, SW1 SW_Push

Commit message: Added optional C7 and fix LED silkscreens
Parts:
- added C7: 100nF, Capacitor_SMD:C_0603_1608Metric, F.Cu at (59.4, 75.1)
- added C7: 100nF, Capacitor_SMD:C_0603_1608Metric, F.Cu at (59.4, 37.0)
- added C7: 100nF, Capacitor_SMD:C_0603_1608Metric, F.Cu at (59.4, 56.1)
- added C7: 100nF, Capacitor_SMD:C_0603_1608Metric, F.Cu at (59.4, 94.2)
- LED1 (x4): value LED -> WS2812B-Mini
