File: poly_kb_atom/poly_kb_molecule_2x1.kicad_pcb (KiCad board)
At the start: 2 copper layers, 38.1 x 19 mm, 76 parts, among them J1 Conn_01x16, J2 North, J3 WestFront, J4 EastFront, J5 WestBack, J6 EastBack, J7 South, J8 North2, J9 South2, SW1 SW_Push

Commit message: Added optional C7 and fix LED silkscreens
Parts:
- added C7: 100nF, Capacitor_SMD:C_0603_1608Metric, F.Cu at (116.6, 56.1)
- added C7: 100nF, Capacitor_SMD:C_0603_1608Metric, F.Cu at (97.5, 56.1)
- LED1 (x2): value LED -> WS2812B-Mini
