File: poly_kb_atom/poly_kb_molecule_4x1_wave_left.kicad_pcb (KiCad board)
At the start: 2 copper layers, 76.2 x 23.8 mm, 95 parts, among them J1 Conn_01x16, J2 North, J3 WestFront, J4 EastFront, J5 WestBack, J6 EastBack, J7 South, J8 North2, J9 South2, SW1 SW_Push

Commit message: Updated remaining molecules and cleanup
Parts:
- added C7: 100nF, Capacitor_SMD:C_0603_1608Metric, F.Cu at (116.8, 53.7)
- added C7: 100nF, Capacitor_SMD:C_0603_1608Metric, F.Cu at (78.7, 53.7)
- added C7: 100nF, Capacitor_SMD:C_0603_1608Metric, F.Cu at (97.7, 51.3)
- added C7: 100nF, Capacitor_SMD:C_0603_1608Metric, F.Cu at (59.6, 56.1)
- J5 (x3): footprint poly_kb:AtomCSInternal -> poly_kb:AtomConnectCS
- LED1 (x4): value LED -> WS2812B-Mini
Routing:
- net CS6: track 93.4 -> 0.00 mm, vias 8 -> 6
- net CS7: track 98.3 -> 191.7 mm, vias 8 -> 10
- net CS5: track 88.6 -> 179.5 mm, vias 8 -> 10
- net CS4: track 90.9 -> 0.00 mm, vias 8 -> 6
- net CS3: track 83.5 -> 167.1 mm, vias 8 -> 10
- net CS2: track 83.7 -> 0.00 mm, vias 8 -> 6
- net CS1: track 79.4 -> 0.00 mm, vias 8 -> 0
- net /Keyboard/sheet605ED2EB/GND: track 162.6 -> 242.0 mm, vias 50 -> 58
