File: poly_kb_atom/poly_kb_molecule_4x1_wave_right.kicad_pcb (KiCad board)
At the start: 2 copper layers, 76.2 x 23.8 mm, 95 parts, among them J1 Conn_01x16, J2 North, J3 WestFront, J4 EastFront, J5 WestBack, J6 EastBack, J7 South, J8 North2, J9 South2, SW1 SW_Push

Commit message: Updated remaining molecules and cleanup
Parts:
- added C7: 100nF, Capacitor_SMD:C_0603_1608Metric, F.Cu at (116.8, 53.7)
- added C7: 100nF, Capacitor_SMD:C_0603_1608Metric, F.Cu at (97.7, 51.3)
- added C7: 100nF, Capacitor_SMD:C_0603_1608Metric, F.Cu at (78.7, 53.7)
- added C7: 100nF, Capacitor_SMD:C_0603_1608Metric, F.Cu at (135.8, 56.1)
- J5 (x3): footprint poly_kb:AtomCSInternal -> poly_kb:AtomConnectCS
- LED1 (x4): value LED -> WS2812B-Mini
Routing:
- net CS7: track 99.1 -> 0.00 mm, vias 8 -> 6
- net CS6: track 93.5 -> 192.6 mm, vias 8 -> 10
- net CS1: track 79.7 -> 0.00 mm, vias 8 -> 0
- net /Keyboard/sheet605ED2EB/GND: track 161.1 -> 240.8 mm, vias 50 -> 58
