File: poly_kb_atom/poly_kb_molecule_4x2_shifted.kicad_pcb (KiCad board)
At the start: 2 copper layers, 85.7 x 38.1 mm, 306 parts, among them J1 Conn_01x16, J2 North, J3 WestFront, J4 EastFront, J5 WestBack, J6 EastBack, J7 South, J8 North2, J9 South2, SW1 SW_Push

Commit message: Updated remaining molecules and cleanup
Parts:
- added C7: 100nF, Capacitor_SMD:C_0603_1608Metric, F.Cu at (145.4, 37.0)
- added C7: 100nF, Capacitor_SMD:C_0603_1608Metric, F.Cu at (107.3, 37.0)
- added C7: 100nF, Capacitor_SMD:C_0603_1608Metric, F.Cu at (154.9, 56.1)
- added C7: 100nF, Capacitor_SMD:C_0603_1608Metric, F.Cu at (135.8, 56.1)
- added C7: 100nF, Capacitor_SMD:C_0603_1608Metric, F.Cu at (97.7, 56.1)
- added C7: 100nF, Capacitor_SMD:C_0603_1608Metric, F.Cu at (88.2, 37.0)
- added C7: 100nF, Capacitor_SMD:C_0603_1608Metric, F.Cu at (126.3, 37.0)
- added C7: 100nF, Capacitor_SMD:C_0603_1608Metric, F.Cu at (116.8, 56.1)
- LED1 (x8): value LED -> WS2812B-Mini
