File: poly_kb_atom/poly_kb_molecule_5x1_wave.kicad_pcb (KiCad board)
At the start: 2 copper layers, 95.2 x 23.8 mm, 114 parts, among them J1 Conn_01x16, J2 North, J3 WestFront, J4 EastFront, J5 WestBack, J6 EastBack, J7 South, J8 North2, J9 South2, SW1 SW_Push

Commit message: Updated remaining molecules and cleanup
Parts:
- added C7: 100nF, Capacitor_SMD:C_0603_1608Metric, F.Cu at (116.8, 53.7)
- added C7: 100nF, Capacitor_SMD:C_0603_1608Metric, F.Cu at (78.7, 53.7)
- added C7: 100nF, Capacitor_SMD:C_0603_1608Metric, F.Cu at (59.6, 56.1)
- added C7: 100nF, Capacitor_SMD:C_0603_1608Metric, F.Cu at (97.7, 51.3)
- added C7: 100nF, Capacitor_SMD:C_0603_1608Metric, F.Cu at (135.8, 56.1)
- J5 (x4): footprint poly_kb:AtomCSInternal -> poly_kb:AtomConnectCS
- LED1 (x5): value LED -> WS2812B-Mini
Routing:
- net CS7: track 124.0 -> 0.00 mm, vias 10 -> 6
- net CS6: track 116.9 -> 240.9 mm, vias 10 -> 14
- net CS5: track 110.8 -> 0.00 mm, vias 10 -> 6
- net CS4: track 113.3 -> 224.1 mm, vias 10 -> 14
- net CS2: track 105.2 -> 0.00 mm, vias 10 -> 6
- net CS3: track 104.8 -> 210.0 mm, vias 10 -> 14
- net CS1: track 99.2 -> 0.00 mm, vias 10 -> 0
- net /Keyboard/sheet605ED2EB/GND: track 202.7 -> 301.9 mm, vias 63 -> 73
