File: poly_kb_atom/ni_buffer.kicad_sch (KiCad schematic)
At the start: 4 parts, among them U31 SN74LVC1G125DCKR, U32 SN74LVC1G125DCKR

Commit message: QFN shift register version
Parts:
- renumbered U31 to U33
Changed lines of the file:
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@@
   (symbol (lib_id "Logic_LevelTranslator:SN74AUP1T34DCK") (at 133.985 135.255 180) (unit 1)
     (in_bom yes) (on_board yes)
-    (property "Reference" "U31" (id 0) (at 130.175 132.715 0))
+    (property "Reference" "U33" (id 0) (at 130.175 132.715 0))
     (property "Value" "SN74LVC1G125DCKR" (id 1) (at 133.985 125.095 0))
     (property "Footprint" "Package_TO_SOT_SMD:SOT-353_SC-70-5" (id 2) (at 133.985 117.475 0)

Commit message: Current production version of right side and added STLs
Parts:
- U32, U33: value SN74LVC1G125DCKR -> 74AHCT1G125SE-7; LCSC C7833 -> (none); MPN SN74LVC1G125DCKR -> C151417
Changed lines of the file:
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@@
     (in_bom yes) (on_board yes)
     (property "Reference" "U32" (id 0) (at 132.715 69.215 0))
-    (property "Value" "SN74LVC1G125DCKR" (id 1) (at 136.525 61.595 0))
+    (property "Value" "74AHCT1G125SE-7" (id 1) (at 136.525 61.595 0))
     (property "Footprint" "Package_TO_SOT_SMD:SOT-353_SC-70-5" (id 2) (at 136.525 53.975 0)
       (effects (font (size 1.27 1.27)) hide)
     )
-    (property "Datasheet" "https://datasheet.lcsc.com/lcsc/1811012330_Texas-Instruments-SN74LVC1G125DCKR_C7833.pdf" (id 3) (at 136.525 56.515 0)
+    (property "Datasheet" "https://datasheet.lcsc.com/lcsc/1912111437_Diodes-Incorporated-74AHCT1G125SE-7_C151417.pdf" (id 3) (at 136.525 56.515 0)
       (effects (font (size 1.27 1.27)) hide)
     )
-    (property "LCSC" "C7833" (id 4) (at 136.525 71.755 0)
+    (property "MPN" "C151417" (id 4) (at 136.525 71.755 0)
       (effects (font (size 1.27 1.27)) hide)
     )
-    (property "MPN" "SN74LVC1G125DCKR" (id 5) (at 136.525 71.755 0)
+    (property "Etc" "" (id 5) (at 136.525 71.755 0)
       (effects (font (size 1.27 1.27)) hide)
     )
@@
     (in_bom yes) (on_board yes)
     (property "Reference" "U33" (id 0) (at 130.175 132.715 0))
-    (property "Value" "SN74LVC1G125DCKR" (id 1) (at 133.985 125.095 0))
+    (property "Value" "74AHCT1G125SE-7" (id 1) (at 133.985 125.095 0))
     (property "Footprint" "Package_TO_SOT_SMD:SOT-353_SC-70-5" (id 2) (at 133.985 117.475 0)
       (effects (font (size 1.27 1.27)) hide)
     )
-    (property "Datasheet" "https://datasheet.lcsc.com/lcsc/1811012330_Texas-Instruments-SN74LVC1G125DCKR_C7833.pdf" (id 3) (at 133.985 120.015 0)
+    (property "Datasheet" "https://datasheet.lcsc.com/lcsc/1912111437_Diodes-Incorporated-74AHCT1G125SE-7_C151417.pdf" (id 3) (at 133.985 120.015 0)
       (effects (font (size 1.27 1.27)) hide)
     )
-    (property "LCSC" "C7833" (id 4) (at 133.985 135.255 0)
+    (property "MPN" "C151417" (id 4) (at 133.985 135.255 0)
       (effects (font (size 1.27 1.27)) hide)
     )
-    (property "MPN" "SN74LVC1G125DCKR" (id 5) (at 133.985 135.255 0)
+    (property "Etc" "" (id 5) (at 133.985 135.255 0)
       (effects (font (size 1.27 1.27)) hide)
     )
