File: poly_kb_atom/shift_registers.kicad_sch (KiCad schematic)
At the start: 5 parts

Commit message: split kb prototype, left side
Parts:
- gave numbers to parts that had none: 5
Connections:
- net Carry4: now reaches U_SR_4.9 (QH'), U_SR_5.14 (SER)
- net Carry2: now reaches U_SR_2.9 (QH'), U_SR_3.14 (SER)
- net Carry3: now reaches U_SR_3.9 (QH'), U_SR_4.14 (SER)
- net Carry1: now reaches U_SR_1.9 (QH'), U_SR_2.14 (SER)
- net Carry renamed CarryOut
- net Reset renamed MReset
Other:
- moved on the sheet: U_SR_1, U_SR_2, U_SR_3, U_SR_4, U_SR_5

Commit message: Final version of wave
Parts:
- U_SR_1, U_SR_2, U_SR_3, U_SR_4, U_SR_5: value 74HCT595 -> (none); footprint Package_SO:SOIC-16_3.9x9.9mm_P1.27mm -> (none); LCSC (none) -> C282339
Changed lines of the file:
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@@
       (effects (font (size 1.27 1.27)) (justify left))
     )
-    (property "Value" "74HCT595" (id 1) (at 259.08 88.9 90)
+    (property "Value" "" (id 1) (at 259.08 88.9 90)
       (effects (font (size 1.27 1.27)) (justify left))
     )
-    (property "Footprint" "Package_SO:SOIC-16_3.9x9.9mm_P1.27mm" (id 2) (at 255.27 90.17 0)
+    (property "Footprint" "" (id 2) (at 255.27 90.17 0)
       (effects (font (size 1.27 1.27)) hide)
     )
     (property "Datasheet" "https://assets.nexperia.com/documents/data-sheet/74HC_HCT595.pdf" (id 3) (at 255.27 90.17 0)
+      (effects (font (size 1.27 1.27)) hide)
+    )
+    (property "LCSC" "C282339" (id 4) (at 255.27 90.17 0)
       (effects (font (size 1.27 1.27)) hide)
     )
@@
       (effects (font (size 1.27 1.27)) (justify left))
     )
-    (property "Value" "74HCT595" (id 1) (at 163.83 88.9 90)
+    (property "Value" "" (id 1) (at 163.83 88.9 90)
       (effects (font (size 1.27 1.27)) (justify left))
     )
-    (property "Footprint" "Package_SO:SOIC-16_3.9x9.9mm_P1.27mm" (id 2) (at 160.02 90.17 0)
+    (property "Footprint" "" (id 2) (at 160.02 90.17 0)
       (effects (font (size 1.27 1.27)) hide)
     )
     (property "Datasheet" "https://assets.nexperia.com/documents/data-sheet/74HC_HCT595.pdf" (id 3) (at 160.02 90.17 0)
+      (effects (font (size 1.27 1.27)) hide)
+    )
+    (property "LCSC" "C282339" (id 4) (at 160.02 90.17 0)
       (effects (font (size 1.27 1.27)) hide)
     )
@@
       (effects (font (size 1.27 1.27)) (justify left))
     )
-    (property "Value" "74HCT595" (id 1) (at 107.95 88.9 90)
+    (property "Value" "" (id 1) (at 107.95 88.9 90)
       (effects (font (size 1.27 1.27)) (justify left))
     )
-    (property "Footprint" "Package_SO:SOIC-16_3.9x9.9mm_P1.27mm" (id 2) (at 104.14 90.17 0)
+    (property "Footprint" "" (id 2) (at 104.14 90.17 0)
       (effects (font (size 1.27 1.27)) hide)
     )
     (property "Datasheet" "https://assets.nexperia.com/documents/data-sheet/74HC_HCT595.pdf" (id 3) (at 104.14 90.17 0)
+      (effects (font (size 1.27 1.27)) hide)
+    )
+    (property "LCSC" "C282339" (id 4) (at 104.14 90.17 0)
       (effects (font (size 1.27 1.27)) hide)
     )
@@
       (effects (font (size 1.27 1.27)) (justify left))
     )
-    (property "Value" "74HCT595" (id 1) (at 57.15 88.9 90)
+    (property "Value" "" (id 1) (at 57.15 88.9 90)
       (effects (font (size 1.27 1.27)) (justify left))
     )
-    (property "Footprint" "Package_SO:SOIC-16_3.9x9.9mm_P1.27mm" (id 2) (at 52.07 90.17 0)
+    (property "Footprint" "" (id 2) (at 52.07 90.17 0)
       (effects (font (size 1.27 1.27)) hide)
     )
     (property "Datasheet" "https://assets.nexperia.com/documents/data-sheet/74HC_HCT595.pdf" (id 3) (at 52.07 90.17 0)
+      (effects (font (size 1.27 1.27)) hide)
+    )
+    (property "LCSC" "C282339" (id 4) (at 52.07 90.17 0)
       (effects (font (size 1.27 1.27)) hide)
     )
@@
       (effects (font (size 1.27 1.27)) (justify left))
     )
-    (property "Value" "74HCT595" (id 1) (at 208.28 88.9 90)
+    (property "Value" "" (id 1) (at 208.28 88.9 90)
       (effects (font (size 1.27 1.27)) (justify left))
     )
-    (property "Footprint" "Package_SO:SOIC-16_3.9x9.9mm_P1.27mm" (id 2) (at 203.2 90.17 0)
+    (property "Footprint" "" (id 2) (at 203.2 90.17 0)
       (effects (font (size 1.27 1.27)) hide)
     )
@@
       (effects (font (size 1.27 1.27)) hide)
     )
+    (property "LCSC" "C282339" (id 4) (at 203.2 90.17 0)
+      (effects (font (size 1.27 1.27)) hide)
+    )

Commit message: Added power leds
Parts:
- U_SR_1, U_SR_2, U_SR_3, U_SR_4, U_SR_5: value (none) -> 74HCT595; JLC (none) -> SOIC-16
Changed lines of the file:
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@@
       (effects (font (size 1.27 1.27)) (justify left))
     )
-    (property "Value" "" (id 1) (at 259.08 88.9 90)
+    (property "Value" "74HCT595" (id 1) (at 259.08 88.9 90)
       (effects (font (size 1.27 1.27)) (justify left))
     )
@@
     )
     (property "LCSC" "C282339" (id 4) (at 255.27 90.17 0)
+      (effects (font (size 1.27 1.27)) hide)
+    )
+    (property "JLC" "SOIC-16" (id 5) (at 255.27 90.17 0)
       (effects (font (size 1.27 1.27)) hide)
     )
@@
       (effects (font (size 1.27 1.27)) (justify left))
     )
-    (property "Value" "" (id 1) (at 163.83 88.9 90)
+    (property "Value" "74HCT595" (id 1) (at 163.83 88.9 90)
       (effects (font (size 1.27 1.27)) (justify left))
     )
@@
     )
     (property "LCSC" "C282339" (id 4) (at 160.02 90.17 0)
+      (effects (font (size 1.27 1.27)) hide)
+    )
+    (property "JLC" "SOIC-16" (id 5) (at 160.02 90.17 0)
       (effects (font (size 1.27 1.27)) hide)
     )
@@
       (effects (font (size 1.27 1.27)) (justify left))
     )
-    (property "Value" "" (id 1) (at 107.95 88.9 90)
+    (property "Value" "74HCT595" (id 1) (at 107.95 88.9 90)
       (effects (font (size 1.27 1.27)) (justify left))
     )
@@
     )
     (property "LCSC" "C282339" (id 4) (at 104.14 90.17 0)
+      (effects (font (size 1.27 1.27)) hide)
+    )
+    (property "JLC" "SOIC-16" (id 5) (at 104.14 90.17 0)
       (effects (font (size 1.27 1.27)) hide)
     )
@@
       (effects (font (size 1.27 1.27)) (justify left))
     )
-    (property "Value" "" (id 1) (at 57.15 88.9 90)
+    (property "Value" "74HCT595" (id 1) (at 57.15 88.9 90)
       (effects (font (size 1.27 1.27)) (justify left))
     )
@@
     )
     (property "LCSC" "C282339" (id 4) (at 52.07 90.17 0)
+      (effects (font (size 1.27 1.27)) hide)
+    )
+    (property "JLC" "SOIC-16" (id 5) (at 52.07 90.17 0)
       (effects (font (size 1.27 1.27)) hide)
     )
@@
       (effects (font (size 1.27 1.27)) (justify left))
     )
-    (property "Value" "" (id 1) (at 208.28 88.9 90)
+    (property "Value" "74HCT595" (id 1) (at 208.28 88.9 90)
       (effects (font (size 1.27 1.27)) (justify left))
     )
@@
       (effects (font (size 1.27 1.27)) hide)
     )
+    (property "JLC" "SOIC-16" (id 5) (at 203.2 90.17 0)
+      (effects (font (size 1.27 1.27)) hide)
+    )

Commit message: Updated WaveL to Revision 1.1
Parts:
- U_SR_1, U_SR_2, U_SR_3, U_SR_4, U_SR_5: footprint (none) -> Package_SO:SOIC-16_3.9x9.9mm_P1.27mm
Changed lines of the file:
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@@
       (effects (font (size 1.27 1.27)) (justify left))
     )
-    (property "Footprint" "" (id 2) (at 255.27 90.17 0)
+    (property "Footprint" "Package_SO:SOIC-16_3.9x9.9mm_P1.27mm" (id 2) (at 255.27 90.17 0)
       (effects (font (size 1.27 1.27)) hide)
     )
@@
       (effects (font (size 1.27 1.27)) (justify left))
     )
-    (property "Footprint" "" (id 2) (at 160.02 90.17 0)
+    (property "Footprint" "Package_SO:SOIC-16_3.9x9.9mm_P1.27mm" (id 2) (at 160.02 90.17 0)
       (effects (font (size 1.27 1.27)) hide)
     )
@@
       (effects (font (size 1.27 1.27)) (justify left))
     )
-    (property "Footprint" "" (id 2) (at 104.14 90.17 0)
+    (property "Footprint" "Package_SO:SOIC-16_3.9x9.9mm_P1.27mm" (id 2) (at 104.14 90.17 0)
       (effects (font (size 1.27 1.27)) hide)
     )
@@
       (effects (font (size 1.27 1.27)) (justify left))
     )
-    (property "Footprint" "" (id 2) (at 52.07 90.17 0)
+    (property "Footprint" "Package_SO:SOIC-16_3.9x9.9mm_P1.27mm" (id 2) (at 52.07 90.17 0)
       (effects (font (size 1.27 1.27)) hide)
     )
@@
       (effects (font (size 1.27 1.27)) (justify left))
     )
-    (property "Footprint" "" (id 2) (at 203.2 90.17 0)
+    (property "Footprint" "Package_SO:SOIC-16_3.9x9.9mm_P1.27mm" (id 2) (at 203.2 90.17 0)
       (effects (font (size 1.27 1.27)) hide)
     )

Commit message: Updated changes made in produced PCB
Parts:
- renumbered U_SR_1 to U4, U_SR_2 to U5, U_SR_3 to U6, U_SR_4 to U7, U_SR_5 to U8
Changed lines of the file:
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@@
   (symbol (lib_id "74xx:74HCT595") (at 255.27 90.17 90) (unit 1)
     (in_bom yes) (on_board yes)
-    (property "Reference" "U_SR_5" (id 0) (at 238.9124 91.3384 90)
+    (property "Reference" "U8" (id 0) (at 256.54 116.84 90)
       (effects (font (size 1.27 1.27)) (justify left))
     )
@@
   (symbol (lib_id "74xx:74HCT595") (at 160.02 90.17 90) (unit 1)
     (in_bom yes) (on_board yes)
-    (property "Reference" "U_SR_3" (id 0) (at 143.6624 91.3384 90)
+    (property "Reference" "U6" (id 0) (at 161.29 116.84 90)
       (effects (font (size 1.27 1.27)) (justify left))
     )
@@
   (symbol (lib_id "74xx:74HCT595") (at 104.14 90.17 90) (unit 1)
     (in_bom yes) (on_board yes)
-    (property "Reference" "U_SR_2" (id 0) (at 87.7824 91.3384 90)
+    (property "Reference" "U5" (id 0) (at 105.41 116.84 90)
       (effects (font (size 1.27 1.27)) (justify left))
     )
@@
   (symbol (lib_id "74xx:74HCT595") (at 52.07 90.17 90) (unit 1)
     (in_bom yes) (on_board yes)
-    (property "Reference" "U_SR_1" (id 0) (at 35.7124 91.3384 90)
+    (property "Reference" "U4" (id 0) (at 53.34 116.84 90)
       (effects (font (size 1.27 1.27)) (justify left))
     )
@@
   (symbol (lib_id "74xx:74HCT595") (at 203.2 90.17 90) (unit 1)
     (in_bom yes) (on_board yes)
-    (property "Reference" "U_SR_4" (id 0) (at 186.8424 91.3384 90)
+    (property "Reference" "U7" (id 0) (at 204.47 116.84 90)
       (effects (font (size 1.27 1.27)) (justify left))
     )

Commit message: Make right side ready
Parts:
- U4, U5, U6, U7, U8: JLC SOIC-16 -> (none); LCSC C282339 -> C2929943; MPN (none) -> 74HC595D
Changed lines of the file:
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@@
       (effects (font (size 1.27 1.27)) hide)
     )
-    (property "Datasheet" "https://assets.nexperia.com/documents/data-sheet/74HC_HCT595.pdf" (id 3) (at 255.27 90.17 0)
+    (property "Datasheet" "https://datasheet.lcsc.com/lcsc/2201121500_Shenzhen-Fuman-Elec-74HC595D-_C2929943.pdf" (id 3) (at 255.27 90.17 0)
       (effects (font (size 1.27 1.27)) hide)
     )
-    (property "LCSC" "C282339" (id 4) (at 255.27 90.17 0)
+    (property "LCSC" "C2929943" (id 4) (at 255.27 90.17 0)
       (effects (font (size 1.27 1.27)) hide)
     )
-    (property "JLC" "SOIC-16" (id 5) (at 255.27 90.17 0)
+    (property "JLC" "" (id 5) (at 255.27 90.17 0)
+      (effects (font (size 1.27 1.27)) hide)
+    )
+    (property "MPN" "74HC595D" (id 6) (at 255.27 90.17 0)
       (effects (font (size 1.27 1.27)) hide)
     )
@@
       (effects (font (size 1.27 1.27)) hide)
     )
-    (property "Datasheet" "https://assets.nexperia.com/documents/data-sheet/74HC_HCT595.pdf" (id 3) (at 160.02 90.17 0)
+    (property "Datasheet" "https://datasheet.lcsc.com/lcsc/2201121500_Shenzhen-Fuman-Elec-74HC595D-_C2929943.pdf" (id 3) (at 160.02 90.17 0)
       (effects (font (size 1.27 1.27)) hide)
     )
-    (property "LCSC" "C282339" (id 4) (at 160.02 90.17 0)
+    (property "LCSC" "C2929943" (id 4) (at 160.02 90.17 0)
       (effects (font (size 1.27 1.27)) hide)
     )
-    (property "JLC" "SOIC-16" (id 5) (at 160.02 90.17 0)
+    (property "JLC" "" (id 5) (at 160.02 90.17 0)
+      (effects (font (size 1.27 1.27)) hide)
+    )
+    (property "MPN" "74HC595D" (id 6) (at 160.02 90.17 0)
       (effects (font (size 1.27 1.27)) hide)
     )
@@
       (effects (font (size 1.27 1.27)) hide)
     )
-    (property "Datasheet" "https://assets.nexperia.com/documents/data-sheet/74HC_HCT595.pdf" (id 3) (at 104.14 90.17 0)
+    (property "Datasheet" "https://datasheet.lcsc.com/lcsc/2201121500_Shenzhen-Fuman-Elec-74HC595D-_C2929943.pdf" (id 3) (at 104.14 90.17 0)
       (effects (font (size 1.27 1.27)) hide)
     )
-    (property "LCSC" "C282339" (id 4) (at 104.14 90.17 0)
+    (property "LCSC" "C2929943" (id 4) (at 104.14 90.17 0)
       (effects (font (size 1.27 1.27)) hide)
     )
-    (property "JLC" "SOIC-16" (id 5) (at 104.14 90.17 0)
+    (property "JLC" "" (id 5) (at 104.14 90.17 0)
+      (effects (font (size 1.27 1.27)) hide)
+    )
+    (property "MPN" "74HC595D" (id 6) (at 104.14 90.17 0)
       (effects (font (size 1.27 1.27)) hide)
     )
@@
       (effects (font (size 1.27 1.27)) hide)
     )
-    (property "Datasheet" "https://assets.nexperia.com/documents/data-sheet/74HC_HCT595.pdf" (id 3) (at 52.07 90.17 0)
+    (property "Datasheet" "https://datasheet.lcsc.com/lcsc/2201121500_Shenzhen-Fuman-Elec-74HC595D-_C2929943.pdf" (id 3) (at 52.07 90.17 0)
       (effects (font (size 1.27 1.27)) hide)
     )
-    (property "LCSC" "C282339" (id 4) (at 52.07 90.17 0)
+    (property "LCSC" "C2929943" (id 4) (at 52.07 90.17 0)
       (effects (font (size 1.27 1.27)) hide)
     )
-    (property "JLC" "SOIC-16" (id 5) (at 52.07 90.17 0)
+    (property "JLC" "" (id 5) (at 52.07 90.17 0)
+      (effects (font (size 1.27 1.27)) hide)
+    )
+    (property "MPN" "74HC595D" (id 6) (at 52.07 90.17 0)
       (effects (font (size 1.27 1.27)) hide)
     )
@@
       (effects (font (size 1.27 1.27)) hide)
     )
-    (property "Datasheet" "https://assets.nexperia.com/documents/data-sheet/74HC_HCT595.pdf" (id 3) (at 203.2 90.17 0)
+    (property "Datasheet" "https://datasheet.lcsc.com/lcsc/2201121500_Shenzhen-Fuman-Elec-74HC595D-_C2929943.pdf" (id 3) (at 203.2 90.17 0)
       (effects (font (size 1.27 1.27)) hide)
     )
-    (property "LCSC" "C282339" (id 4) (at 203.2 90.17 0)
+    (property "LCSC" "C2929943" (id 4) (at 203.2 90.17 0)
       (effects (font (size 1.27 1.27)) hide)
     )
-    (property "JLC" "SOIC-16" (id 5) (at 203.2 90.17 0)
+    (property "JLC" "" (id 5) (at 203.2 90.17 0)
       (effects (font (size 1.27 1.27)) hide)
     )
+    (property "MPN" "74HC595D" (id 6) (at 203.2 90.17 0)
+      (effects (font (size 1.27 1.27)) hide)
+    )
