File: poly_kb_atom/ni_buffer2.kicad_sch (KiCad schematic)
At the start: 2 parts, among them U14 SN74LVC1G126DBVR, U15 SN74LVC1G126DBVR

Commit message: Updated all openSCAD models and various fixes for the right side before final production
Parts:
- U14, U15: MPN C7834 -> C151890
Connections:
- net GND: now also U14.1 (VCCA), U15.1 (VCCA)
- net VCC: no longer U14.1 (VCCA), U15.1 (VCCA)
Changed lines of the file:
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@@
     (effects (font (size 1.27 1.27)) (justify left bottom))
   )
-  (hierarchical_label "VCC" (shape input) (at 139.065 151.13 270) (fields_autoplaced)
+  (hierarchical_label "GND" (shape input) (at 139.065 151.13 270) (fields_autoplaced)
     (effects (font (size 1.27 1.27)) (justify right))
   )
@@
     (effects (font (size 1.27 1.27)) (justify left))
   )
+  (hierarchical_label "GND" (shape input) (at 139.065 87.63 270) (fields_autoplaced)
+    (effects (font (size 1.27 1.27)) (justify right))
+  )
   (hierarchical_label "GND" (shape input) (at 136.525 113.665 90) (fields_autoplaced)
     (effects (font (size 1.27 1.27)) (justify left))
-  )
-  (hierarchical_label "VCC" (shape input) (at 139.065 87.63 270) (fields_autoplaced)
-    (effects (font (size 1.27 1.27)) (justify right))
   )
   (hierarchical_label "VCC" (shape input) (at 133.985 151.13 270) (fields_autoplaced)
@@
       (effects (font (size 1.27 1.27)) hide)
     )
-    (property "Datasheet" "http://www.ti.com/lit/ds/symlink/sn74aup1t34.pdf" (at 136.525 56.515 0)
+    (property "Datasheet" "https://www.ti.com/cn/lit/gpn/sn74ahc1g125" (at 136.525 56.515 0)
       (effects (font (size 1.27 1.27)) hide)
     )
-    (property "MPN" "C7834" (at 136.525 71.755 0)
+    (property "MPN" "C151890" (at 136.525 71.755 0)
       (effects (font (size 1.27 1.27)) hide)
     )
@@
         )
         (path "/e63e39d7-6ac0-4ffd-8aa3-1841a4541b55/4f637138-78e8-4078-835b-92e3f188adc0"
-          (reference "U11") (unit 1)
+          (reference "U12") (unit 1)
         )
         (path "/e63e39d7-6ac0-4ffd-8aa3-1841a4541b55/cc4e6829-8f50-4fc4-85c0-49f5930ba461"
@@
       (effects (font (size 1.27 1.27)) hide)
     )
-    (property "Datasheet" "http://www.ti.com/lit/ds/symlink/sn74aup1t34.pdf" (at 136.525 120.015 0)
+    (property "Datasheet" "https://www.ti.com/cn/lit/gpn/sn74ahc1g125" (at 136.525 120.015 0)
       (effects (font (size 1.27 1.27)) hide)
     )
-    (property "MPN" "C7834" (at 136.525 135.255 0)
+    (property "MPN" "C151890" (at 136.525 135.255 0)
       (effects (font (size 1.27 1.27)) hide)
     )
@@
         )
         (path "/e63e39d7-6ac0-4ffd-8aa3-1841a4541b55/4f637138-78e8-4078-835b-92e3f188adc0"
-          (reference "U12") (unit 1)
+          (reference "U13") (unit 1)
         )
         (path "/e63e39d7-6ac0-4ffd-8aa3-1841a4541b55/cc4e6829-8f50-4fc4-85c0-49f5930ba461"
