File: poly_kb_atom/poly_kb_wave_left2.kicad_sch (KiCad schematic)
At the start: 47 parts, among them J37 FH34SRJ-12S-0.5SH, J38 Conn_01x05, J39 FH12-30S-0.5SH, SW1 RotaryEncoder_Switch, U2 TD6811, U3 MT9700

Commit message: Added revision 2.2 and latest STLs
Connections:
- net Col8: no longer SW1.C
- net GND: now also SW1.C
- no-connect marks 14 -> 15
