File: poly_kb_atom/poly_kb_wave_right2.kicad_sch (KiCad schematic)
At the start: 46 parts, among them J37 FH34SRJ-12S-0.5SH, J38 Conn_01x05, J39 FH12-30S-0.5SH, SW1 RotaryEncoder_Switch, U2 TD6811, U3 MT9700

Commit message: Revised Rev2
Parts:
- added R25: 5.1K 0402, Resistor_SMD:R_0402_1005Metric, symbol Device:R_Small
Connections:
- net GND: now also R25.1; no longer R13.2
- net VBUS: no longer C10.1, U2.4 (VDD)
- net VSYS: now also C10.1, U2.4 (VDD)
- new net: R13.2, R25.2
Other:
- note added: "Increase for more current: Imax = 6.8k / RSet"
- note added: "RSet"
- note added: "~250mA Max"
- note removed: "300mA Max"
- note removed: "Increase for more current: Imax = 6.8k / R13"

Commit message: Right side: Production version Rev2
Parts:
- C33, C34: value 4.7uF Tantalum -> 4.7uF 3216 25V Tantalum
- D5: value Green 0805 -> Green 0805 C2297
- D6: value Yellow 0805 -> Yellow 0805 C2296
- J37: footprint poly_kb:FH34SRJ12S05SH50 -> poly_kb:FH34SRJ12S05SH50-Rev2
Other:
- title: PolyKB Wave R -> PolyKB PacificWave R
Changed lines of the file:
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@@
   (paper "A2")
   (title_block
-    (title "PolyKB Wave R")
+    (title "PolyKB PacificWave R")
     (rev "2")
   )
@@
     (effects (font (size 3 3) (thickness 0.6) bold) (justify left bottom))
   )
-  (text "~250mA Max" (at 540.385 349.25 0)
+  (text "~250mA Max" (at 554.99 349.25 0)
     (effects (font (size 1.27 1.27)) (justify left bottom))
   )
@@
     (effects (font (size 1.27 1.27)) (justify left bottom))
   )
+  (label "VBAT" (at 322.58 198.755 0) (fields_autoplaced)
+    (effects (font (size 1.27 1.27)) (justify left bottom))
+  )
   (label "SDIN4" (at 212.09 76.835 0) (fields_autoplaced)
     (effects (font (size 1.27 1.27)) (justify left bottom))
@@
       (effects (font (size 1.27 1.27)) (justify left))
     )
-    (property "Value" "10uF 0805 16V" (at 537.21 355.6 0)
+    (property "Value" "10uF 0805 16V" (at 539.115 349.25 0)
       (effects (font (size 1.27 1.27)) (justify left))
     )
@@
       (effects (font (size 1.27 1.27)) (justify right))
     )
-    (property "Value" "Green 0805" (at 556.26 355.6 90)
+    (property "Value" "Green 0805 C2297" (at 549.275 356.235 90)
       (effects (font (size 1.27 1.27)) (justify right))
     )
@@
       (effects (font (size 1.27 1.27)) hide)
     )
-    (property "JLC" "" (at 554.99 353.06 0)
-      (effects (font (size 1.27 1.27)) hide)
-    )
     (property "MPN" "C2297" (at 554.99 353.06 0)
       (effects (font (size 1.27 1.27)) hide)
@@
       (effects (font (size 1.27 1.27)) (justify right))
     )
-    (property "Value" "4.7uF Tantalum" (at 442.595 306.705 90)
+    (property "Value" "4.7uF 3216 25V Tantalum" (at 442.595 306.705 90)
       (effects (font (size 1.27 1.27)) (justify right))
     )
@@
       (effects (font (size 1.27 1.27)))
     )
-    (property "JLC" "" (at 447.04 306.705 0)
-      (effects (font (size 1.27 1.27)) hide)
-    )
-    (property "Etc" "" (at 447.04 306.705 0)
-      (effects (font (size 1.27 1.27)) hide)
-    )
     (pin "1")
     (pin "2")
@@
       (effects (font (size 1.27 1.27)))
     )
-    (property "Footprint" "poly_kb:FH34SRJ12S05SH50" (at 549.275 125.73 0)
+    (property "Footprint" "poly_kb:FH34SRJ12S05SH50-Rev2" (at 549.275 125.73 0)
       (effects (font (size 1.27 1.27)) hide)
     )
@@
       (effects (font (size 1.27 1.27)) (justify right))
     )
-    (property "Value" "Yellow 0805" (at 555.625 309.1814 90)
+    (property "Value" "Yellow 0805 C2296" (at 555.625 309.1814 90)
       (effects (font (size 1.27 1.27)) (justify right))
     )
@@
       (effects (font (size 1.27 1.27)) hide)
     )
-    (property "JLC" "" (at 553.085 307.975 0)
-      (effects (font (size 1.27 1.27)) hide)
-    )
     (property "MPN" "C2296" (at 553.085 307.975 0)
       (effects (font (size 1.27 1.27)) hide)
@@
       (effects (font (size 1.27 1.27)) (justify right))
     )
-    (property "Value" "4.7uF Tantalum" (at 456.565 306.07 90)
+    (property "Value" "4.7uF 3216 25V Tantalum" (at 456.565 306.07 90)
       (effects (font (size 1.27 1.27)) (justify right))
     )

Commit message: Updated all openSCAD models and various fixes for the right side before final production
Parts:
- SW1: footprint poly_kb:EVQWGD001_ALPS-EC11_mod -> poly_kb:PolyJog
- renumbered JP3 to JP1
Connections:
- net VBAT: no longer C2.1, J39.6 (Pin_6)
- net VDD: now also C2.1, J39.6 (Pin_6)
Other:
- note added: "VBAT current limit (display array and LED matrix)"
- note removed: "Display Array Current Limiter 3V3"
- title: PolyKB PacificWave R -> PolyKybd Split R
- moved on the sheet: DBG3
Changed lines of the file:
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@@
   (paper "A2")
   (title_block
-    (title "PolyKB PacificWave R")
+    (title "PolyKybd Split R")
+    (date "2023-03-09")
     (rev "2")
   )
@@
     (effects (font (size 3 3) (thickness 0.6) bold) (justify left bottom))
   )
-  (text "Display Array Current Limiter 3V3" (at 481.965 342.9 0)
+  (text "VBAT current limit (display array and LED matrix)" (at 466.09 341.63 0)
     (effects (font (size 3 3) (thickness 0.6) bold) (justify left bottom))
   )
@@
     )
   )
-  (global_label "SR_DATA" (shape input) (at 424.815 67.31 0) (fields_autoplaced)
+  (global_label "SR_DATA" (shape input) (at 551.815 35.56 0) (fields_autoplaced)
     (effects (font (size 1.27 1.27)) (justify left))
-    (property "Intersheetrefs" "${INTERSHEET_REFS}" (at 435.09 67.3894 0)
+    (property "Intersheetrefs" "${INTERSHEET_REFS}" (at 562.09 35.6394 0)
       (effects (font (size 1.27 1.27)) (justify left) hide)
     )
@@
     )
   )
-  (global_label "D-C" (shape input) (at 424.815 74.93 0) (fields_autoplaced)
+  (global_label "D-C" (shape input) (at 551.815 43.18 0) (fields_autoplaced)
     (effects (font (size 1.27 1.27)) (justify left))
-    (property "Intersheetrefs" "${INTERSHEET_REFS}" (at 431.3405 75.0094 0)
+    (property "Intersheetrefs" "${INTERSHEET_REFS}" (at 558.3405 43.2594 0)
       (effects (font (size 1.27 1.27)) (justify left) hide)
     )
@@
     )
   )
-  (global_label "SERIAL_COM1" (shape input) (at 478.79 185.42 180) (fields_autoplaced)
-    (effects (font (size 1.27 1.27)) (justify right))
-    (property "Intersheetrefs" "${INTERSHEET_REFS}" (at 463.7979 185.3406 0)
-      (effects (font (size 1.27 1.27)) (justify right) hide)
-    )
-  )
   (global_label "Col5" (shape input) (at 500.38 223.52 180) (fields_autoplaced)
     (effects (font (size 1.27 1.27)) (justify right))
@@
     )
   )
-  (global_label "SR_LATCH" (shape input) (at 424.815 64.77 0) (fields_autoplaced)
+  (global_label "SR_LATCH" (shape input) (at 551.815 33.02 0) (fields_autoplaced)
     (effects (font (size 1.27 1.27)) (justify left))
-    (property "Intersheetrefs" "${INTERSHEET_REFS}" (at 436.36 64.8494 0)
+    (property "Intersheetrefs" "${INTERSHEET_REFS}" (at 563.36 33.0994 0)
       (effects (font (size 1.27 1.27)) (justify left) hide)
     )
@@
     )
   )
-  (global_label "VDD" (shape input) (at 424.815 62.23 0) (fields_autoplaced)
+  (global_label "VDD" (shape input) (at 551.815 30.48 0) (fields_autoplaced)
     (effects (font (size 1.27 1.27)) (justify left))
-    (property "Intersheetrefs" "${INTERSHEET_REFS}" (at 436.1786 62.1506 0)
+    (property "Intersheetrefs" "${INTERSHEET_REFS}" (at 563.1786 30.4006 0)
       (effects (font (size 1.27 1.27)) (justify left) hide)
     )
@@
     )
   )
-  (global_label "VBAT" (shape input) (at 424.815 59.69 0) (fields_autoplaced)
+  (global_label "VBAT" (shape input) (at 551.815 27.94 0) (fields_autoplaced)
     (effects (font (size 1.27 1.27)) (justify left))
-    (property "Intersheetrefs" "${INTERSHEET_REFS}" (at 436.9648 59.6106 0)
+    (property "Intersheetrefs" "${INTERSHEET_REFS}" (at 563.9648 27.8606 0)
       (effects (font (size 1.27 1.27)) (justify left) hide)
     )
@@
     )
   )
-  (global_label "VBAT" (shape input) (at 393.7 325.755 270) (fields_autoplaced)
-    (effects (font (size 1.27 1.27)) (justify right))
-    (property "Intersheetrefs" "${INTERSHEET_REFS}" (at 393.7794 337.9048 90)
-      (effects (font (size 1.27 1.27)) (justify right) hide)
-    )
-  )
   (global_label "SR_CLOCK" (shape input) (at 554.355 185.42 0) (fields_autoplaced)
     (effects (font (size 1.27 1.27)) (justify left))
@@
     )
   )
-  (global_label "SDIN_RAW" (shape input) (at 424.815 77.47 0) (fields_autoplaced)
+  (global_label "SDIN_RAW" (shape input) (at 551.815 45.72 0) (fields_autoplaced)
     (effects (font (size 1.27 1.27)) (justify left))
-    (property "Intersheetrefs" "${INTERSHEET_REFS}" (at 436.4205 77.3906 0)
+    (property "Intersheetrefs" "${INTERSHEET_REFS}" (at 563.4205 45.6406 0)
       (effects (font (size 1.27 1.27)) (justify left) hide)
     )
@@
     )
   )
-  (global_label "SR_CLOCK" (shape input) (at 424.815 69.85 0) (fields_autoplaced)
+  (global_label "SR_CLOCK" (shape input) (at 551.815 38.1 0) (fields_autoplaced)
     (effects (font (size 1.27 1.27)) (justify left))
-    (property "Intersheetrefs" "${INTERSHEET_REFS}" (at 436.8438 69.9294 0)
+    (property "Intersheetrefs" "${INTERSHEET_REFS}" (at 563.8438 38.1794 0)
       (effects (font (size 1.27 1.27)) (justify left) hide)
     )
   )
+  (global_label "VDD" (shape input) (at 393.7 325.755 270) (fields_autoplaced)
+    (effects (font (size 1.27 1.27)) (justify right))
+    (property "Intersheetrefs" "${INTERSHEET_REFS}" (at 393.7794 337.1186 90)
+      (effects (font (size 1.27 1.27)) (justify right) hide)
+    )
+  )
   (global_label "SCLK_RAW" (shape input) (at 439.42 193.04 180) (fields_autoplaced)
     (effects (font (size 1.27 1.27)) (justify right))
@@
     )
   )
-  (global_label "SCLK_RAW" (shape input) (at 424.815 80.01 0) (fields_autoplaced)
+  (global_label "SCLK_RAW" (shape input) (at 551.815 48.26 0) (fields_autoplaced)
     (effects (font (size 1.27 1.27)) (justify left))
-    (property "Intersheetrefs" "${INTERSHEET_REFS}" (at 436.7833 79.9306 0)
+    (property "Intersheetrefs" "${INTERSHEET_REFS}" (at 563.7833 48.1806 0)
       (effects (font (size 1.27 1.27)) (justify left) hide)
     )
@@
     )
   )
-  (global_label "RESET" (shape input) (at 424.815 72.39 0) (fields_autoplaced)
+  (global_label "RESET" (shape input) (at 551.815 40.64 0) (fields_autoplaced)
     (effects (font (size 1.27 1.27)) (justify left))
-    (property "Intersheetrefs" "${INTERSHEET_REFS}" (at 432.9733 72.4694 0)
+    (property "Intersheetrefs" "${INTERSHEET_REFS}" (at 559.9733 40.7194 0)
       (effects (font (size 1.27 1.27)) (justify left) hide)
     )
@@
     )
   )
-  (global_label "GND" (shape input) (at 424.815 82.55 0) (fields_autoplaced)
+  (global_label "GND" (shape input) (at 551.815 50.8 0) (fields_autoplaced)
     (effects (font (size 1.27 1.27)) (justify left))
-    (property "Intersheetrefs" "${INTERSHEET_REFS}" (at 431.0986 82.6294 0)
+    (property "Intersheetrefs" "${INTERSHEET_REFS}" (at 558.0986 50.8794 0)
       (effects (font (size 1.27 1.27)) (justify left) hide)
     )
@@
     )
   )
+  (global_label "SERIAL_COM1" (shape input) (at 478.79 185.42 180) (fields_autoplaced)
+    (effects (font (size 1.27 1.27)) (justify right))
+    (property "Intersheetrefs" "${INTERSHEET_REFS}" (at 463.3052 185.42 0)
+      (effects (font (size 1.27 1.27)) (justify right) hide)
+    )
+  )
   (global_label "D-C" (shape input) (at 239.395 33.02 0) (fields_autoplaced)
     (effects (font (size 1.27 1.27)) (justify left))
@@
     )
   )
-  (symbol (lib_id "Connector_Generic:Conn_01x10") (at 419.735 72.39 180) (unit 1)
+  (symbol (lib_id "Connector_Generic:Conn_01x10") (at 546.735 40.64 180) (unit 1)
     (in_bom yes) (on_board yes) (dnp no) (fields_autoplaced)
-    (property "Reference" "DBG3" (at 419.735 52.705 0)
+    (property "Reference" "DBG3" (at 546.735 20.955 0)
       (effects (font (size 1.27 1.27)))
     )
-    (property "Value" "DebugPort" (at 419.735 55.245 0)
+    (property "Value" "DebugPort" (at 546.735 23.495 0)
       (effects (font (size 1.27 1.27)))
     )
-    (property "Footprint" "Connector_PinHeader_2.54mm:PinHeader_1x10_P2.54mm_Vertical" (at 419.735 72.39 0)
+    (property "Footprint" "Connector_PinHeader_2.54mm:PinHeader_1x10_P2.54mm_Vertical" (at 546.735 40.64 0)
       (effects (font (size 1.27 1.27)) hide)
     )
-    (property "Datasheet" "~" (at 419.735 72.39 0)
+    (property "Datasheet" "~" (at 546.735 40.64 0)
       (effects (font (size 1.27 1.27)) hide)
     )
@@
       (effects (font (size 1.27 1.27)))
     )
-    (property "Footprint" "poly_kb:EVQWGD001_ALPS-EC11_mod" (at 38.735 201.041 0)
+    (property "Footprint" "poly_kb:PolyJog" (at 38.735 201.041 0)
       (effects (font (size 1.27 1.27)) hide)
     )
@@
   (symbol (lib_id "Jumper:SolderJumper_3_Bridged12") (at 568.96 350.52 0) (unit 1)
     (in_bom yes) (on_board yes) (dnp no)
-    (property "Reference" "JP3" (at 567.69 343.535 0)
+    (property "Reference" "JP1" (at 567.69 343.535 0)
       (effects (font (size 1.27 1.27)) (justify left))
     )
@@
       (project "poly_kb_wave_right2"
         (path "/e63e39d7-6ac0-4ffd-8aa3-1841a4541b55"
-          (reference "JP3") (unit 1)
+          (reference "JP1") (unit 1)
         )
       )

Commit message: Added revision 2.2 and latest STLs
Connections:
- net Col1: no longer SW1.C
- net GND: now also SW1.C
Other:
- title: PolyKybd Split R -> PolyKybd Split72 R
Changed lines of the file:
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@@
   (paper "A2")
   (title_block
-    (title "PolyKybd Split R")
-    (date "2023-03-09")
-    (rev "2")
+    (title "PolyKybd Split72 R")
+    (date "2023-06-22")
+    (rev "2.2")
   )
   (junction (at 259.08 219.075) (diameter 0) (color 0 0 0 0)
@@
     (stroke (width 0) (type default))
   )
-  (wire (pts (xy 33.655 205.105) (xy 33.655 216.535))
-    (stroke (width 0) (type default))
-  )
   (wire (pts (xy 106.68 18.415) (xy 128.905 18.415))
     (stroke (width 0) (type default))
@@
     (stroke (width 0) (type default))
   )
-  (wire (pts (xy 33.655 216.535) (xy 50.165 216.535))
-    (stroke (width 0) (type default))
-  )
   (bus (pts (xy 104.14 28.575) (xy 104.14 31.115))
     (stroke (width 0) (type default))
@@
     )
   )
+  (global_label "GND" (shape input) (at 33.655 205.105 180) (fields_autoplaced)
+    (effects (font (size 1.27 1.27)) (justify right))
+    (property "Intersheetrefs" "${INTERSHEET_REFS}" (at 26.8787 205.105 0)
+      (effects (font (size 1.27 1.27)) (justify right) hide)
+    )
+  )
   (global_label "GND" (shape input) (at 411.48 296.545 270) (fields_autoplaced)
     (effects (font (size 1.27 1.27)) (justify right))
@@
     )
   )
-  (global_label "Col1" (shape input) (at 33.655 216.535 270) (fields_autoplaced)
+  (global_label "Col1" (shape input) (at 50.165 216.535 270) (fields_autoplaced)
     (effects (font (size 1.27 1.27)) (justify right))
-    (property "Intersheetrefs" "${INTERSHEET_REFS}" (at 33.5756 223.2419 90)
+    (property "Intersheetrefs" "${INTERSHEET_REFS}" (at 50.0856 223.2419 90)
       (effects (font (size 1.27 1.27)) (justify right) hide)
     )
