File: poly_kybd/poly_kybd_split72_left.kicad_sch (KiCad schematic)
At the start: 48 parts, among them J37 FH34SRJ-12S-0.5SH, J38 Conn_01x05, J39 FH12-30S-0.5SH, SW1 RotaryEncoder_Switch, U2 TLV62569DBVR, U26 TPD4E05U06DQAR, U3 SY6280AAC

Commit message: Added rev 3.2 for right side
Parts:
- U2: footprint Package_TO_SOT_SMD:TSOT-23-5 -> Package_TO_SOT_SMD:SOT-23-5
Changed lines of the file:
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@@
 			)
 		)
-		(property "Footprint" "Package_TO_SOT_SMD:TSOT-23-5"
+		(property "Footprint" "Package_TO_SOT_SMD:SOT-23-5"
 			(at 508.635 286.385 0)
 			(effects
