File: poly_kybd/poly_kybd_split72_left.kicad_sch (KiCad schematic)
At the start: 48 parts, among them J37 FH34SRJ-12S-0.5SH, J38 Conn_01x05, J39 FH12-30S-0.5SH, SW1 RotaryEncoder_Switch, U2 TLV62569DBVR, U26 TPD4E05U06DQAR, U3 SY6280AAC

Commit message: A5: replace four EOL parts across schematics, PCBs and the project library
All four were discontinued at JLCPCB ("no longer manufactured", 0 stock),
so the v3.2 BOM can no longer be ordered as-is. Metadata only - every
replacement keeps the same footprint, so no layout or netlist changes.

  C118249  Sunlord  TC212A475K025Y  -> C5380411 Vishay  293D475X9025A2TE3
  C170128  Samsung  CL10C6R8DB8NNNC -> C318672  Samsung CL10C6R8CB8NNNC
  C3303719 Nexperia 74HC595BQ115    -> C730243  Nexperia 74HC595BQ,115
  C2940195 Winbond  W25Q64JVXGIQ    -> C5440778 Winbond W25Q64JVXGIM

Net cost at a 200-keyboard batch: -$4.15/keyboard, -$829/batch. The flash
carries it (-$4.76/kbd); the tantalum is the only real increase
(+$0.68/kbd, and it was the only 4.7uF/25V CASE-A with volume).

Also fixed along the way:

- MPN held the LCSC code rather than a manufacturer part number on all
  four, the same defect as the buffer in #24. Now the real MPN.
- The 74HC595 datasheet pointed at a rocelec.widen.net mirror that is now
  404. Repointed to Nexperia's own copy, verified to be the
  74HC595/74HCT595 data sheet. That URL was in poly_kb.kicad_sym too, so
  the project library and its cached copies are updated together.
- Manufacturer "winbond" -> "Winbond", "Sunlord" -> "Vishay".

Scope: the corne split42 variant shares these parts and is included -
leaving EOL codes anywhere is a trap. Library and footprint identifiers
containing "XGIQ" (lib_id, sym-lib-table path, footprint name, search
tags) are deliberately unchanged: they are names, not part numbers, and
renaming them would break the library binding.

Verified: 422 property edits across 14 files, insertions and deletions
exactly balanced, and every changed line is a (property ...) line - no
pads, nets, placements or reference designators touched.

Co-Authored-By: Claude Opus 5 <noreply@anthropic.com>
Parts:
- C11: JLC C170128 -> C318672; LCSC C170128 -> C318672; MPN C170128 -> CL10C6R8CB8NNNC
- C33, C34: JLC C118249 -> C5380411; LCSC C118249 -> C5380411; MPN C118249 -> 293D475X9025A2TE3; Manufacturer Sunlord -> Vishay
Changed lines of the file:
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@@
 			)
 		)
-		(property "Datasheet" "https://www.lcsc.com/datasheet/lcsc_datasheet_1810010229_CEC-Shenzhen-Zhenhua-XinYun-Elec-CA45-A-25V-4-7uF-K_C129569.pdf"
+		(property "Datasheet" "https://www.vishay.com/docs/40002/293d.pdf"
 			(at 447.04 306.705 0)
 			(effects
@@
 			)
 		)
-		(property "MPN" "C118249"
+		(property "MPN" "293D475X9025A2TE3"
 			(at 439.42 313.055 90)
 			(effects
@@
 			)
 		)
-		(property "JLC" "C118249"
+		(property "JLC" "C5380411"
 			(at 447.04 306.705 0)
 			(effects
@@
 			)
 		)
-		(property "LCSC" "C118249"
+		(property "LCSC" "C5380411"
 			(at 447.04 306.705 0)
 			(effects
@@
 			)
 		)
-		(property "Manufacturer" "Sunlord"
+		(property "Manufacturer" "Vishay"
 			(at 447.04 306.705 0)
 			(effects
@@
 			)
 		)
-		(property "Datasheet" "https://www.lcsc.com/datasheet/lcsc_datasheet_1810010229_CEC-Shenzhen-Zhenhua-XinYun-Elec-CA45-A-25V-4-7uF-K_C129569.pdf"
+		(property "Datasheet" "https://www.vishay.com/docs/40002/293d.pdf"
 			(at 449.58 311.785 0)
 			(effects
@@
 			)
 		)
-		(property "MPN" "C118249"
+		(property "MPN" "293D475X9025A2TE3"
 			(at 452.755 315.595 90)
 			(effects
@@
 			)
 		)
-		(property "JLC" "C118249"
+		(property "JLC" "C5380411"
 			(at 449.58 311.785 0)
 			(effects
@@
 			)
 		)
-		(property "LCSC" "C118249"
+		(property "LCSC" "C5380411"
 			(at 449.58 311.785 0)
 			(effects
@@
 			)
 		)
-		(property "Manufacturer" "Sunlord"
+		(property "Manufacturer" "Vishay"
 			(at 449.58 311.785 0)
 			(effects
@@
 			)
 		)
-		(property "Datasheet" "https://www.lcsc.com/datasheet/lcsc_datasheet_2304140030_Samsung-Electro-Mechanics-CL10C6R8DB8NNNC_C170128.pdf"
+		(property "Datasheet" "https://wmsc.lcsc.com/wmsc/upload/file/pdf/v2/lcsc/2304140030_Samsung-Electro-Mechanics-CL10C6R8CB8NNNC_C318672.pdf"
 			(at 534.035 300.355 0)
 			(effects
@@
 			)
 		)
-		(property "MPN" "C170128"
+		(property "MPN" "CL10C6R8CB8NNNC"
 			(at 534.035 300.355 0)
 			(effects
@@
 			)
 		)
-		(property "JLC" "C170128"
+		(property "JLC" "C318672"
 			(at 534.035 300.355 0)
 			(effects
@@
 			)
 		)
-		(property "LCSC" "C170128"
+		(property "LCSC" "C318672"
 			(at 534.035 300.355 0)
 			(effects
