File: poly_kybd/SSD1306_TO_SPI_NO_LED.kicad_sch (KiCad schematic)
At the start: 11 parts, among them J1 FH34SRJ-14S-0.5SH

Commit message: misc updates (including missing for corne split42)
Parts:
- removed LED1: XL-3030RGBC, poly_kb:XL-3030RGBC-WS2812B, symbol LED:WS2812B
Other:
- title: Display Adapter, LED & Switch -> Display Adapter & Switch
