File: poly_kybd/ni_buffer2.kicad_sch (KiCad schematic)
At the start: 2 parts, among them U14 SN74LVC1G126DBVR, U15 SN74LVC1G126DBVR

Commit message: Revision D caps and schematics part cleanup
Parts:
- U14, U15: JLC (none) -> C151890; LCSC (none) -> C151890
Changed lines of the file:
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@@
+      (effects (font (size 1.27 1.27)) hide)
+    )
+    (property "JLC" "C151890" (at 136.525 71.755 0)
+      (effects (font (size 1.27 1.27)) hide)
+    )
+    (property "LCSC" "C151890" (at 136.525 71.755 0)
       (effects (font (size 1.27 1.27)) hide)
     )
@@
       (effects (font (size 1.27 1.27)) hide)
     )
+    (property "JLC" "C151890" (at 136.525 135.255 0)
+      (effects (font (size 1.27 1.27)) hide)
+    )
+    (property "LCSC" "C151890" (at 136.525 135.255 0)
+      (effects (font (size 1.27 1.27)) hide)
+    )

Commit message: Updated left side for RoHS
Parts:
- U14, U15: Manufacturer (none) -> TI; RoHS (none) -> x
Changed lines of the file:
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@@
+      (effects (font (size 1.27 1.27)) hide)
+    )
+    (property "Manufacturer" "TI" (at 136.525 71.755 0)
+      (effects (font (size 1.27 1.27)) hide)
+    )
+    (property "RoHS" "x" (at 136.525 71.755 0)
       (effects (font (size 1.27 1.27)) hide)
     )
@@
       (effects (font (size 1.27 1.27)) hide)
     )
+    (property "Manufacturer" "TI" (at 136.525 135.255 0)
+      (effects (font (size 1.27 1.27)) hide)
+    )
+    (property "RoHS" "x" (at 136.525 135.255 0)
+      (effects (font (size 1.27 1.27)) hide)
+    )

Commit message: Renamed schematics and pcb files; cleanup; Updated left side to 3.2; Added submodules
Parts:
- renumbered U14 to U20, U15 to U21

Commit message: misc updates (including missing for corne split42)
Parts:
- renumbered U20 to U12, U21 to U13
Changed lines of the file:
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@@
 (kicad_sch
-	(version 20231120)
+	(version 20250114)
 	(generator "eeschema")
-	(generator_version "8.0")
+	(generator_version "9.0")
 	(paper "A4")
-	(wire
-		(pts
-			(xy 136.525 50.165) (xy 136.525 64.135)
-		)
-		(stroke
-			(width 0)
-			(type default)
-		)
-	)
-	(wire
-		(pts
-			(xy 139.065 79.375) (xy 139.065 87.63)
-		)
-		(stroke
-			(width 0)
-			(type default)
-		)
-	)
-	(wire
-		(pts
-			(xy 139.065 142.875) (xy 139.065 151.13)
-		)
-		(stroke
-			(width 0)
-			(type default)
-		)
-	)
-	(wire
-		(pts
-			(xy 118.745 71.755) (xy 126.365 71.755)
-		)
-		(stroke
-			(width 0)
-			(type default)
-		)
-	)
-	(wire
-		(pts
-			(xy 133.985 142.875) (xy 133.985 151.13)
-		)
-		(stroke
-			(width 0)
-			(type default)
-		)
-	)
-	(wire
-		(pts
-			(xy 133.985 79.375) (xy 133.985 87.63)
-		)
-		(stroke
-			(width 0)
-			(type default)
-		)
-	)
-	(wire
-		(pts
-			(xy 136.525 113.665) (xy 136.525 127.635)
-		)
-		(stroke
-			(width 0)
-			(type default)
-		)
-	)
-	(wire
-		(pts
-			(xy 118.745 135.255) (xy 126.365 135.255)
-		)
-		(stroke
-			(width 0)
-			(type default)
-		)
-	)
-	(wire
-		(pts
-			(xy 146.685 71.755) (xy 156.845 71.755)
-		)
-		(stroke
-			(width 0)
-			(type default)
-		)
-	)
-	(wire
-		(pts
-			(xy 146.685 135.255) (xy 156.845 135.255)
-		)
-		(stroke
-			(width 0)
-			(type default)
-		)
-	)
 	(text "Output Enable"
 		(exclude_from_sim no)
@@
 		)
 	)
+	(wire
+		(pts
+			(xy 136.525 50.165) (xy 136.525 64.135)
+		)
+		(stroke
+			(width 0)
+			(type default)
+		)
+	)
+	(wire
+		(pts
+			(xy 139.065 79.375) (xy 139.065 87.63)
+		)
+		(stroke
+			(width 0)
+			(type default)
+		)
+	)
+	(wire
+		(pts
+			(xy 139.065 142.875) (xy 139.065 151.13)
+		)
+		(stroke
+			(width 0)
+			(type default)
+		)
+	)
+	(wire
+		(pts
+			(xy 118.745 71.755) (xy 126.365 71.755)
+		)
+		(stroke
+			(width 0)
+			(type default)
+		)
+	)
+	(wire
+		(pts
+			(xy 133.985 142.875) (xy 133.985 151.13)
+		)
+		(stroke
+			(width 0)
+			(type default)
+		)
+	)
+	(wire
+		(pts
+			(xy 133.985 79.375) (xy 133.985 87.63)
+		)
+		(stroke
+			(width 0)
+			(type default)
+		)
+	)
+	(wire
+		(pts
+			(xy 136.525 113.665) (xy 136.525 127.635)
+		)
+		(stroke
+			(width 0)
+			(type default)
+		)
+	)
+	(wire
+		(pts
+			(xy 118.745 135.255) (xy 126.365 135.255)
+		)
+		(stroke
+			(width 0)
+			(type default)
+		)
+	)
+	(wire
+		(pts
+			(xy 146.685 71.755) (xy 156.845 71.755)
+		)
+		(stroke
+			(width 0)
+			(type default)
+		)
+	)
+	(wire
+		(pts
+			(xy 146.685 135.255) (xy 156.845 135.255)
+		)
+		(stroke
+			(width 0)
+			(type default)
+		)
+	)
 	(hierarchical_label "GND"
 		(shape input)
 		(at 139.065 151.13 270)
-		(fields_autoplaced yes)
 		(effects
 			(font
@@
 		(shape input)
 		(at 118.745 135.255 180)
-		(fields_autoplaced yes)
 		(effects
 			(font
@@
 		(shape input)
 		(at 118.745 71.755 180)
-		(fields_autoplaced yes)
 		(effects
 			(font
@@
 		(shape input)
 		(at 136.525 50.165 90)
-		(fields_autoplaced yes)
 		(effects
 			(font
@@
 		(shape input)
 		(at 133.985 87.63 270)
-		(fields_autoplaced yes)
 		(effects
 			(font
@@
 		(shape input)
 		(at 156.845 135.255 0)
-		(fields_autoplaced yes)
 		(effects
 			(font
@@
 		(shape input)
 		(at 139.065 87.63 270)
-		(fields_autoplaced yes)
 		(effects
 			(font
@@
 		(shape input)
 		(at 136.525 113.665 90)
-		(fields_autoplaced yes)
 		(effects
 			(font
@@
 		(shape input)
 		(at 133.985 151.13 270)
-		(fields_autoplaced yes)
 		(effects
 			(font
@@
 		(shape input)
 		(at 156.845 71.755 0)
-		(fields_autoplaced yes)
 		(effects
 			(font
@@
 		(on_board yes)
 		(dnp no)
-		(property "Reference" "U20"
+		(property "Reference" "U12"
 			(at 132.715 69.215 0)
 			(effects
@@
 		)
 		(instances
-			(project "poly_kb_wave_left2"
+			(project "poly_corne_split42_left"
 				(path "/e63e39d7-6ac0-4ffd-8aa3-1841a4541b55/340f60e4-2ba5-4a69-be5b-84823556915d"
 					(reference "U20")
@@
 				)
 				(path "/e63e39d7-6ac0-4ffd-8aa3-1841a4541b55/b3eec1c7-cfcb-457c-8bc1-731941cd757b"
-					(reference "U24")
+					(reference "U?")
 					(unit 1)
 				)
@@
 		(on_board yes)
 		(dnp no)
-		(property "Reference" "U21"
+		(property "Reference" "U13"
 			(at 132.715 132.715 0)
 			(effects
@@
 		)
 		(instances
-			(project "poly_kb_wave_left2"
+			(project "poly_corne_split42_left"
 				(path "/e63e39d7-6ac0-4ffd-8aa3-1841a4541b55/340f60e4-2ba5-4a69-be5b-84823556915d"
 					(reference "U21")
@@
 				)
 				(path "/e63e39d7-6ac0-4ffd-8aa3-1841a4541b55/b3eec1c7-cfcb-457c-8bc1-731941cd757b"
-					(reference "U25")
-					(unit 1)
-				)
+					(reference "U?")
+					(unit 1)
+				)
