File: poly_kybd/poly_kybd_split72_right.kicad_sch (KiCad schematic)
At the start: 47 parts, among them J37 FH34SRJ-12S-0.5SH, J38 Conn_01x05, J39 FH12-30S-0.5SH, SW1 RotaryEncoder_Switch, U2 TD6811, U3 MT9700

Commit message: Added rev 3.2 for right side
Parts:
- added U26: TPD4E05U06DQAR, poly_kb:USON-10, symbol acheron_Symbols:TPD4E05U06DQAR
- C10: value 10uF 0805 16V -> 4.7uF 0805 25V; JLC (none) -> C1779; LCSC (none) -> C1779; MPN C15850 -> C1779; Manufacturer (none) -> Samsung; RoHS (none) -> x
- C11: value 22pF 0603 16V -> 6.8pF 0603 50V; JLC (none) -> C170128; LCSC (none) -> C170128; MPN C1653 -> C170128; Manufacturer (none) -> Samsung; RoHS (none) -> x
- C12, C13, C14: JLC (none) -> C15850; LCSC (none) -> C15850; Manufacturer (none) -> Samsung; RoHS (none) -> x
- C2, C30, C31, C32: JLC (none) -> C52923; LCSC (none) -> C52923; Manufacturer (none) -> Samsung; RoHS (none) -> x
- C33, C34: Etc (none) -> Preorder Req; JLC (none) -> C118249; LCSC (none) -> C118249; MPN C129569 -> C118249; Manufacturer (none) -> Sunlord; RoHS (none) -> x
- D12: value 1N4148WS -> 1N4148WSX; JLC (none) -> C6423741; LCSC (none) -> C6423741; MPN C2128 -> C6423741; Manufacturer (none) -> Shenzhen JingYang; RoHS (none) -> x
- D5: JLC (none) -> C2297; LCSC (none) -> C2297; Manufacturer (none) -> Hubei KENTO; RoHS (none) -> x
- D6: JLC (none) -> C2296; LCSC (none) -> C2296; Manufacturer (none) -> Hubei KENTO; RoHS (none) -> x
- DBG1, DBG3, H1, H2, H3, H4, H5, H6, H7, H8, H9, J38, JP1, SW1: JLC (none) -> DNP; LCSC (none) -> DNP; MPN (none) -> DNP
- FB2: JLC (none) -> C1017; LCSC (none) -> C1017; Manufacturer (none) -> Sunlord; RoHS (none) -> x
- J37: JLC (none) -> C424659; LCSC (none) -> C424659; Manufacturer (none) -> Hirose; RoHS (none) -> x
- J39: JLC (none) -> C506793; LCSC (none) -> C506793; Manufacturer (none) -> Hirose; RoHS (none) -> x
- L1: value 4.7uH -> 2.2uH; footprint poly_kb:MCS0530-4R7MN2 -> poly_kb:SMMS0420-2R2M; JLC (none) -> C133191; LCSC (none) -> C133191; MPN C2836880 -> C133191; Manufacturer (none) -> SXN; RoHS (none) -> x
- R1, R2: JLC (none) -> C108405; LCSC (none) -> C108405; MPN C23345 -> C108405; Manufacturer (none) -> Yageo; RoHS (none) -> x
- R10, R11: value 390k 0603 -> 390k 0603 1%; JLC (none) -> C137735; LCSC (none) -> C137735; MPN C23150 -> C137735; Manufacturer (none) -> Yageo; RoHS (none) -> x
- R12: JLC (none) -> C114660; LCSC (none) -> C114660; MPN C22807 -> C114660; Manufacturer (none) -> Yageo; RoHS (none) -> x
- R13: JLC C22790 -> C114659; LCSC (none) -> C114659; MPN C22790 -> C114659; Manufacturer (none) -> Yageo; RoHS (none) -> x
- R25: value 10K 0402 -> 10k 0402; JLC (none) -> C60490; LCSC (none) -> C60490; MPN C25744 -> C60490; Manufacturer (none) -> Yageo; RoHS (none) -> x
- R3, R4: JLC (none) -> C144745; LCSC (none) -> C144745; MPN C25905 -> C144745; Manufacturer (none) -> Yageo; RoHS (none) -> x
- R30: JLC (none) -> C137735; LCSC (none) -> C137735; MPN C23150 -> C137735; Manufacturer (none) -> Yageo; RoHS (none) -> x
- R5, R6: value 1k 0603 -> 1k 0402; footprint Resistor_SMD:R_0603_1608Metric -> Resistor_SMD:R_0402_1005Metric; JLC (none) -> C144789; LCSC (none) -> C144789; MPN C21190 -> C144789; Manufacturer (none) -> Yageo; RoHS (none) -> x
- U2: value TD6811 -> TLV62569DBVR; footprint Package_TO_SOT_SMD:TSOT-23-5 -> Package_TO_SOT_SMD:SOT-23-5; Etc (none) -> Replaced C189486 with C141836 (TI) (alt C222072 (ST)); JLC (none) -> C141836; LCSC (none) -> C141836; MPN C189486 -> C141836; Manufacturer (none) -> TI; RoHS (none) -> x
- U3: value MT9700 -> SY6280AAC; JLC (none) -> C55136; LCSC (none) -> C55136; MPN C89855 -> C55136; Manufacturer (none) -> Silergy; RoHS (none) -> x
- USB2: JLC (none) -> C165948; LCSC (none) -> C165948; Manufacturer (none) -> Hroparts; RoHS (none) -> x
Connections:
- net GND: now also U26.3 (GND), U26.8 (GND)
- net SERIAL_COM1: now also U26.1 (IO1), U26.10 (NC), U26.4 (D2+), U26.7 (NC)
- net SERIAL_COM2: now also U26.2 (IO2), U26.5 (D2-), U26.6 (NC), U26.9 (NC)
Other:
- moved on the sheet: FB2, USB2
