File: poly_kybd/poly_kybd_split72_right.kicad_sch (KiCad schematic)
At the start: 48 parts, among them J37 FH34SRJ-12S-0.5SH, J38 Conn_01x05, J39 FH12-30S-0.5SH, SW1 RotaryEncoder_Switch, U2 TLV62569DBVR, U26 TPD4E05U06DQAR, U3 SY6280AAC

Commit message: 1k 0402: retarget from Yageo C144789 to Vishay C71623
C144789 (Yageo AC0402FR-071KL) is not being restocked, and its remaining
listing carries a minimum purchase of 3,445 pieces against the 2,000
needed for a 200-keyboard batch.

Vishay CRCW04021K00FKED (C71623) is an exact functional match:

                   Yageo C144789      Vishay C71623
  value/package    1k 0402            1k 0402
  tolerance        +-1%               +-1%
  TCR              +-100ppm/C         +-100ppm/C
  power            62.5 mW            63 mW
  temperature      -55..+155 C        -55..+155 C
  stock            12,804 (min 3445)  374,486 (min 1)

Costs $0.0038 against $0.0029, so +$1.80 across a 200-keyboard batch.

R5, R6, R16, R19, R21 - 5 per board, on all four boards and in the
schematics (rp_pico.kicad_sch is shared, so its R16/R19/R21 serve every
project). 31 instances, 155 field edits.

MPN also corrected: it held the LCSC code rather than a manufacturer part
number, the same defect fixed on the buffer in #24. Datasheet repointed to
Vishay's own copy rather than an LCSC mirror.

No new RoHS evidence needed: the part carries Vishay's "e3" lead-free
termination code, and vishay-rohs-20250901.pdf - added for the tantalum -
is a company-wide statement covering all Vishay products.

Scoped strictly on JLC/LCSC == C144789, never on Manufacturer == Yageo:
212 other footprint fields on these boards are also Yageo and are
untouched. In particular AC0402FR-075K1L (the 5.1k, R3/R4/R7/R9) is a
different part in the same series and is unchanged.

Every changed line is a (property ...) line. Footprint, placement, pads
and net assignments asserted identical before and after.

Co-Authored-By: Claude Opus 5 <noreply@anthropic.com>
Parts:
- R5, R6: JLC C144789 -> C71623; LCSC C144789 -> C71623; MPN C144789 -> CRCW04021K00FKED; Manufacturer Yageo -> Vishay
Changed lines of the file:
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@@
 			)
 		)
-		(property "Datasheet" "https://www.lcsc.com/datasheet/lcsc_datasheet_2304140030_YAGEO-AC0402FR-071KL_C144789.pdf"
+		(property "Datasheet" "https://www.vishay.com/docs/20035/dcrcwe3.pdf"
 			(at 554.355 359.41 0)
 			(effects
@@
 			)
 		)
-		(property "MPN" "C144789"
+		(property "MPN" "CRCW04021K00FKED"
 			(at 554.355 359.41 0)
 			(effects
@@
 			)
 		)
-		(property "JLC" "C144789"
+		(property "JLC" "C71623"
 			(at 554.355 359.41 0)
 			(effects
@@
 			)
 		)
-		(property "LCSC" "C144789"
+		(property "LCSC" "C71623"
 			(at 554.355 359.41 0)
 			(effects
@@
 			)
 		)
-		(property "Manufacturer" "Yageo"
+		(property "Manufacturer" "Vishay"
 			(at 554.355 359.41 0)
 			(effects
@@
 			)
 		)
-		(property "Datasheet" "https://www.lcsc.com/datasheet/lcsc_datasheet_2304140030_YAGEO-AC0402FR-071KL_C144789.pdf"
+		(property "Datasheet" "https://www.vishay.com/docs/20035/dcrcwe3.pdf"
 			(at 551.18 316.23 0)
 			(effects
@@
 			)
 		)
-		(property "MPN" "C144789"
+		(property "MPN" "CRCW04021K00FKED"
 			(at 551.18 316.23 0)
 			(effects
@@
 			)
 		)
-		(property "JLC" "C144789"
+		(property "JLC" "C71623"
 			(at 551.18 316.23 0)
 			(effects
@@
 			)
 		)
-		(property "LCSC" "C144789"
+		(property "LCSC" "C71623"
 			(at 551.18 316.23 0)
 			(effects
@@
 			)
 		)
-		(property "Manufacturer" "Yageo"
+		(property "Manufacturer" "Vishay"
 			(at 551.18 316.23 0)
 			(effects

Commit message: USB-C: bring HRO-TYPE-C-31-M-12-Assembly into poly_kb.pretty, repoint the schematics
The EnvUSB library (thirdparty/EnvOpenPico/.../HRO-TYPE-C31-M-12.pretty) is not
in this repo, so KiCad reports it missing on open. It was the only one of the
eight missing footprint libraries genuinely in use - the other seven are dead
references, and Nexperia595 turned out to be vestigial too, appearing only in a
lib_symbols cache while all nine 74HC595 instances already use poly_kb.

Nothing was broken, because the footprint is embedded in all four boards, but
Update PCB from Schematic could not resolve it - which is exactly what the
coming layout pass needs. Since it was embedded, it could be recovered from the
tree rather than hunted upstream: extracted from poly_kybd_split72_left USB1 and
stripped of instance-only data (42 uuids, 1 sheet path, 16 pad nets, the
placement, the USB1 reference).

Validated rather than assumed: parens balanced 300/300, 14 distinct pad names
with geometry identical to the board, 13 graphic elements kept, and the board
instance carried no descr or 3D model, so nothing was lost.

Kept on B.Cu deliberately. All eight instances across the four boards are
bottom-mounted, so there is no front-side instance to copy, and keeping the
as-built side avoids a front/back mirroring transformation that has no
reference to verify against - the failure mode there is a silently mirrored
connector. The provenance and this reasoning are recorded in the footprint's
descr.

Schematics: 5 instances repointed from EnvUSB: to poly_kb: - USB1 in
rp_pico.kicad_sch and USB2 in both split72 and both split42 top sheets. No
lib_symbols cache carried the reference, so none had to be touched.

The boards still name EnvUSB: for the placed footprints. That is inert - the
geometry is embedded and identical - and the next Update PCB from Schematic
will swap them to the poly_kb name.

Co-Authored-By: Claude Opus 5 <noreply@anthropic.com>
Claude-Session: https://claude.ai/code/session_013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
Parts:
- USB2: footprint EnvUSB:HRO-TYPE-C-31-M-12-Assembly -> poly_kb:HRO-TYPE-C-31-M-12-Assembly
Changed lines of the file:
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@@
 			)
 		)
-		(property "Footprint" "EnvUSB:HRO-TYPE-C-31-M-12-Assembly"
+		(property "Footprint" "poly_kb:HRO-TYPE-C-31-M-12-Assembly"
 			(at 402.59 348.996 0)
 			(effects
