File: poly_kybd/rp_pico.kicad_sch (KiCad schematic)
At the start: 47 parts, among them SW2 EVQPUC02K, SW3 EVQPUC02K, U10 RP2040, U11 TPD4E05U06DQAR, U2 TD6811, U9 W25Q64JVXGIQ, Y1 TAXM12M4RFBCCT2T

Commit message: Update PCB and plate to rev3 (disconnected vbus via bridge and removed polyfuse)
Parts:
- removed D2: ESD5Z5V0, Diode_SMD:D_SOD-523, symbol Diode:SMF6V0A
- removed F1: 2920L030DR, Fuse:Fuse_2920_7451Metric, symbol Device:Fuse
- added D2: 1N5819WS, poly_kb:D_SOD-323Ext, symbol Device:D_Schottky_Small
Connections:
- net VBUS: now also R8.1, D2.2 (A)
- net VSYS: now also D2.1 (K); no longer R8.1
Other:
- note removed: "IHold = 300mA, ITrip = 600 mA"
- note removed: "If USB is the only power source it is safe to use VBUS=VSYS, otherwise we need no insert a Schottky barrier diode in-between."
- moved on the sheet: R15, R8

Commit message: Added latest gerber files, latest STLs and updated readme
Parts:
- R24: MPN C22938 -> C170723

Commit message: Revision D caps and schematics part cleanup
Parts:
- C15, C16, C17, C18, C19, C20, C21, C22, C23, C9: JLC (none) -> C1525; LCSC (none) -> C1525
- C24, C25: JLC (none) -> C52923; LCSC (none) -> C52923
- C26, C4, C6: JLC (none) -> C15850; LCSC (none) -> C15850
- C3, C8: JLC (none) -> C1557; LCSC (none) -> C1557
- C5: JLC (none) -> C1653; LCSC (none) -> C1653
- D1: JLC (none) -> C84256; LCSC (none) -> C84256
- D2: JLC (none) -> C191023; LCSC (none) -> C191023
- FB1: JLC (none) -> C1017; LCSC (none) -> C1017
- L2: JLC (none) -> C2836880; LCSC (none) -> C2836880
- R14: JLC (none) -> C25822; LCSC (none) -> C25822
- R15, R20: JLC (none) -> C25744; LCSC (none) -> C25744
- R16, R19: JLC (none) -> C21190; LCSC (none) -> C21190
- R17: JLC (none) -> C22807; LCSC (none) -> C22807
- R18: JLC (none) -> C7250; LCSC (none) -> C7250
- R21: JLC (none) -> C11702; LCSC (none) -> C11702
- R22, R23: JLC (none) -> C25190; LCSC (none) -> C25190
- R24: JLC (none) -> C170723; LCSC (none) -> C170723
- R7, R9: JLC (none) -> C25905; LCSC (none) -> C25905
- R8: JLC (none) -> C25908; LCSC (none) -> C25908
- SW2, SW3: JLC (none) -> C79174; LCSC (none) -> C79174
- TP1, TP14: JLC (none) -> DNP; LCSC (none) -> DNP; MPN (none) -> DNP
- U10: JLC (none) -> C2040; LCSC (none) -> C2040
- U11: JLC (none) -> C2836386; LCSC (none) -> C2836386
- U2: JLC (none) -> C189486; LCSC (none) -> C189486
- U9: JLC (none) -> C2940195; LCSC (none) -> C2940195
- USB1: JLC (none) -> C165948; LCSC (none) -> C165948
- Y1: JLC (none) -> C133337; LCSC (none) -> C133337

Commit message: Updated left side for RoHS
Parts:
- removed C4: 10uF 0805 16V, Capacitor_SMD:C_0805_2012Metric, symbol Device:C_Small
- removed C5: 22pF 0603 16V, Capacitor_SMD:C_0603_1608Metric, symbol Device:C_Small
- removed L2: 4.7uH, poly_kb:MCS0530-4R7MN2, symbol Device:L
- added C10: 4.7uF 0805 25V, Capacitor_SMD:C_0805_2012Metric, symbol Device:C_Small
- added C11: 6.8pF 0603 50V, Capacitor_SMD:C_0603_1608Metric, symbol Device:C_Small
- added L1: 2.2uH, poly_kb:SMMS0420-2R2M, symbol Device:L
- C15, C16, C17, C18, C19, C20, C21, C22, C23, C6, C9: Manufacturer (none) -> Samsung; RoHS (none) -> x
- C24, C25: value 1uf 0402 16V -> 1uF 0402 16V; Manufacturer (none) -> Samsung; RoHS (none) -> x
- C26: value 10uf 0805 16V -> 10uF 0805 16V; Manufacturer (none) -> Samsung; RoHS (none) -> x
- C3, C8: Manufacturer (none) -> FH; RoHS (none) -> x
- D1: Manufacturer (none) -> NationStar; RoHS (none) -> x
- D2: Etc (none) -> C5278927 is RoHS / Paker; Manufacturer (none) -> Hottech Semi; RoHS (none) -> x Email sent
- FB1: Manufacturer (none) -> Sunlord; RoHS (none) -> x
- R14: JLC C25822 -> C137690; LCSC C25822 -> C137690; MPN C25822 -> C137690; Manufacturer (none) -> Yageo; RoHS (none) -> x
- R15, R20: value 10K 0402 -> 10k 0402; JLC C25744 -> C60490; LCSC C25744 -> C60490; MPN C25744 -> C60490; Manufacturer (none) -> Yageo; RoHS (none) -> x
- R16, R19: value 1k 0603 -> 1k 0402; footprint Resistor_SMD:R_0603_1608Metric -> Resistor_SMD:R_0402_1005Metric; JLC C21190 -> C144789; LCSC C21190 -> C144789; MPN C21190 -> C144789; Manufacturer (none) -> Yageo; RoHS (none) -> x
- R17: JLC C22807 -> C114660; LCSC C22807 -> C114660; MPN C22807 -> C114660; Manufacturer (none) -> Yageo; RoHS (none) -> x
- R18: JLC C7250 -> C141675; LCSC C7250 -> C141675; MPN C7250 -> C141675; Manufacturer (none) -> Yageo; RoHS (none) -> x
- R21: value 1K 0402 -> 1k 0402; JLC C11702 -> C144789; LCSC C11702 -> C144789; MPN C11702 -> C144789; Manufacturer (none) -> Yageo; RoHS (none) -> x
- R22, R23: JLC C25190 -> C137753; LCSC C25190 -> C137753; MPN C25190 -> C137753; Manufacturer (none) -> Yageo; RoHS (none) -> x
- R24: JLC C170723 -> C137747; LCSC C170723 -> C137747; MPN C170723 -> C137747; Manufacturer (none) -> Yageo; RoHS (none) -> x
- R7, R9: JLC C25905 -> C144745; LCSC C25905 -> C144745; MPN C25905 -> C144745; Manufacturer (none) -> Yageo; RoHS (none) -> x
- R8: JLC C25908 -> C163457; LCSC C25908 -> C163457; MPN C25908 -> C163457; Manufacturer (none) -> Yageo; RoHS (none) -> x
- SW2, SW3: Etc (none) -> Low Stock; Manufacturer (none) -> Panasonic; RoHS (none) -> x
- U10: Manufacturer (none) -> Raspberry Pi; RoHS (none) -> x
- U11: Manufacturer (none) -> MSKSEMI; RoHS (none) -> x
- U2: value TD6811 -> TLV62569DBVR; Etc (none) -> Replaced C189486 with C141836 (TI) (alt C222072 (ST)); JLC C189486 -> C141836; LCSC C189486 -> C141836; MPN C189486 -> C141836; Manufacturer (none) -> TI; RoHS (none) -> x
- U9: Manufacturer (none) -> winbond; RoHS (none) -> x
- USB1: Manufacturer (none) -> Hroparts; RoHS (none) -> x
- Y1: value TAXM12M4RFBCCT2T -> 7M12000044; JLC C133337 -> C93114; LCSC C133337 -> C93114; MPN C133337 -> C93114; Manufacturer (none) -> TXC; RoHS (none) -> x
Connections:
- net 3V3: now also C11.1, L1.2
- net GND: now also C10.2
- net VSYS: now also C10.1
- net at U2.3 (SW): now also L1.1
- net at R14.1, R17.2, R18.1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: now also C11.2

Commit message: Renamed schematics and pcb files; cleanup; Updated left side to 3.2; Added submodules
Parts:
- U9: footprint SON80P400X400X50-9N -> poly_kb:DFN_XGIQ TR_WIN
- renumbered C10 to C4, C11 to C5, L1 to L2, U2 to U1

Commit message: Added rev 3.2 for right side
Parts:
- U1: footprint Package_TO_SOT_SMD:TSOT-23-5 -> Package_TO_SOT_SMD:SOT-23-5
Changed lines of the file:
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@@
 			)
 		)
-		(property "Footprint" "Package_TO_SOT_SMD:TSOT-23-5"
+		(property "Footprint" "Package_TO_SOT_SMD:SOT-23-5"
 			(at 213.36 40.005 0)
 			(effects

Commit message: misc updates (including missing for corne split42)
Parts:
- C3, C8: JLC C1557 -> C86287; LCSC C1557 -> C86287; MPN C1557 -> C86287; Manufacturer FH -> Samsung
- D2: Etc C5278927 is RoHS / Paker -> (none); Manufacturer Hottech Semi -> Hottech; RoHS x Email sent -> x
