File: poly_kybd/rp_pico.kicad_sch (KiCad schematic)
At the start: 46 parts, among them SW2 EVQPUC02K, SW3 EVQPUC02K, U1 TLV62569DBVR, U10 RP2040, U11 TPD4E05U06DQAR, U9 W25Q64JVXGIM, Y1 7M12000044

Commit message: 1k 0402: retarget from Yageo C144789 to Vishay C71623
C144789 (Yageo AC0402FR-071KL) is not being restocked, and its remaining
listing carries a minimum purchase of 3,445 pieces against the 2,000
needed for a 200-keyboard batch.

Vishay CRCW04021K00FKED (C71623) is an exact functional match:

                   Yageo C144789      Vishay C71623
  value/package    1k 0402            1k 0402
  tolerance        +-1%               +-1%
  TCR              +-100ppm/C         +-100ppm/C
  power            62.5 mW            63 mW
  temperature      -55..+155 C        -55..+155 C
  stock            12,804 (min 3445)  374,486 (min 1)

Costs $0.0038 against $0.0029, so +$1.80 across a 200-keyboard batch.

R5, R6, R16, R19, R21 - 5 per board, on all four boards and in the
schematics (rp_pico.kicad_sch is shared, so its R16/R19/R21 serve every
project). 31 instances, 155 field edits.

MPN also corrected: it held the LCSC code rather than a manufacturer part
number, the same defect fixed on the buffer in #24. Datasheet repointed to
Vishay's own copy rather than an LCSC mirror.

No new RoHS evidence needed: the part carries Vishay's "e3" lead-free
termination code, and vishay-rohs-20250901.pdf - added for the tantalum -
is a company-wide statement covering all Vishay products.

Scoped strictly on JLC/LCSC == C144789, never on Manufacturer == Yageo:
212 other footprint fields on these boards are also Yageo and are
untouched. In particular AC0402FR-075K1L (the 5.1k, R3/R4/R7/R9) is a
different part in the same series and is unchanged.

Every changed line is a (property ...) line. Footprint, placement, pads
and net assignments asserted identical before and after.

Co-Authored-By: Claude Opus 5 <noreply@anthropic.com>
Parts:
- R16, R19, R21: JLC C144789 -> C71623; LCSC C144789 -> C71623; MPN C144789 -> CRCW04021K00FKED; Manufacturer Yageo -> Vishay
Changed lines of the file:
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@@
 			)
 		)
-		(property "Datasheet" "https://www.lcsc.com/datasheet/lcsc_datasheet_2304140030_YAGEO-AC0402FR-071KL_C144789.pdf"
+		(property "Datasheet" "https://www.vishay.com/docs/20035/dcrcwe3.pdf"
 			(at 261.62 70.485 0)
 			(effects
@@
 			)
 		)
-		(property "MPN" "C144789"
+		(property "MPN" "CRCW04021K00FKED"
 			(at 261.62 70.485 0)
 			(effects
@@
 			)
 		)
-		(property "JLC" "C144789"
+		(property "JLC" "C71623"
 			(at 261.62 70.485 0)
 			(effects
@@
 			)
 		)
-		(property "LCSC" "C144789"
+		(property "LCSC" "C71623"
 			(at 261.62 70.485 0)
 			(effects
@@
 			)
 		)
-		(property "Manufacturer" "Yageo"
+		(property "Manufacturer" "Vishay"
 			(at 261.62 70.485 0)
 			(effects
@@
 			)
 		)
-		(property "Datasheet" "https://www.lcsc.com/datasheet/lcsc_datasheet_2304140030_YAGEO-AC0402FR-071KL_C144789.pdf"
+		(property "Datasheet" "https://www.vishay.com/docs/20035/dcrcwe3.pdf"
 			(at 346.71 78.74 0)
 			(effects
@@
 			)
 		)
-		(property "MPN" "C144789"
+		(property "MPN" "CRCW04021K00FKED"
 			(at 346.71 78.74 0)
 			(effects
@@
 			)
 		)
-		(property "JLC" "C144789"
+		(property "JLC" "C71623"
 			(at 346.71 78.74 0)
 			(effects
@@
 			)
 		)
-		(property "LCSC" "C144789"
+		(property "LCSC" "C71623"
 			(at 346.71 78.74 0)
 			(effects
@@
 			)
 		)
-		(property "Manufacturer" "Yageo"
+		(property "Manufacturer" "Vishay"
 			(at 346.71 78.74 0)
 			(effects
@@
 			)
 		)
-		(property "Datasheet" "https://www.lcsc.com/datasheet/lcsc_datasheet_2304140030_YAGEO-AC0402FR-071KL_C144789.pdf"
+		(property "Datasheet" "https://www.vishay.com/docs/20035/dcrcwe3.pdf"
 			(at 33.02 229.235 0)
 			(effects
@@
 			)
 		)
-		(property "MPN" "C144789"
+		(property "MPN" "CRCW04021K00FKED"
 			(at 33.02 229.235 0)
 			(effects
@@
 			)
 		)
-		(property "JLC" "C144789"
+		(property "JLC" "C71623"
 			(at 33.02 229.235 0)
 			(effects
@@
 			)
 		)
-		(property "LCSC" "C144789"
+		(property "LCSC" "C71623"
 			(at 33.02 229.235 0)
 			(effects
@@
 			)
 		)
-		(property "Manufacturer" "Yageo"
+		(property "Manufacturer" "Vishay"
 			(at 33.02 229.235 0)
 			(effects

Commit message: U9 -> Boya BY25Q64ESCIG(R), RGB LEDs -> XINGLIGHT XL-3332RGBC
Schematic-only. Both parts change package, so neither is a running change and
the layout work is NOT in this commit.

U9 (rp_pico.kicad_sch): Winbond W25Q64JVXGIM C5440778 -> BOYAMICRO
BY25Q64ESCIG(R) C50176394, quoted $0.6012 x 400 = $240.48 at 7 business days,
with a RoHS certificate already filed. Package goes 4x4 DFN -> LGA-8 2x3, so
the footprint moves to the KiCad stock Package_SON:SON-8-1EP_3x2mm_P0.5mm_
EP1.4x1.6mm. The symbol is kept: the pinout is an 8/8 match to the nets already
on U9, so it is electrically right - only its library name still says Winbond.

LED1 (SSD1306_TO_SPI.kicad_sch, the shared sheet, so all 72 instances follow):
XL-3030RGBC C5349958 -> XL-3332RGBC C42400839, $1.48/kbd against $4.43, i.e.
-$2.85/kbd or -$570 per 200-unit batch. The lens change is now free because the
diffuser frame spreads the light, which is what retired the bench test that had
blocked this.

Adds poly_kb.pretty/XL-3332RGBC-WS2812B.kicad_mod. Two warnings carried in the
footprint's own descr field, because they are load-bearing:

- The land pattern is UNVERIFIED. Unlike the XL-3030RGBC, this datasheet has no
  Recommended Soldering Pattern page - only a package outline. The pads here are
  the datasheet terminal bands (VDD full-width top 0.65, GND full-width bottom
  0.65, DI/DO side blocks 1.10 x 0.80, 1.00 centre column) plus a 0.20 mm toe
  extension outward, inner edges untouched so the gaps are preserved.
- The terminal topology is nothing like the 3030's four corner pads, so this is
  a re-route at 72 positions rather than a pad swap, and DI/DO handedness comes
  from reading the top and bottom views against each other. Verify both against
  a physical sample or a vendor drawing before fabrication.

Co-Authored-By: Claude Opus 5 <noreply@anthropic.com>
Claude-Session: https://claude.ai/code/session_013TdVkG4xm84QHBhBEYQUBe
Parts:
- U9: value W25Q64JVXGIM -> BY25Q64ESCIG(R); footprint poly_kb:DFN_XGIQ TR_WIN -> Package_SON:SON-8-1EP_3x2mm_P0.5mm_EP1.4x1.6mm; JLC C5440778 -> C50176394; LCSC C5440778 -> C50176394; MPN W25Q64JVXGIM -> BY25Q64ESCIG(R); Manufacturer Winbond -> BOYAMICRO
Changed lines of the file:
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@@
 			)
 		)
-		(property "Value" "W25Q64JVXGIM"
+		(property "Value" "BY25Q64ESCIG(R)"
 			(at 76.2 224.79 0)
 			(effects
@@
 			)
 		)
-		(property "Footprint" "poly_kb:DFN_XGIQ TR_WIN"
+		(property "Footprint" "Package_SON:SON-8-1EP_3x2mm_P0.5mm_EP1.4x1.6mm"
 			(at 100.33 226.695 0)
 			(effects
@@
 			)
 		)
-		(property "Datasheet" "https://www.winbond.com/resource-files/W25Q64JV%20RevK%2003102021%20Plus.pdf"
+		(property "Datasheet" "https://www.lcsc.com/product-detail/C50176394.html"
 			(at 100.33 229.235 0)
 			(effects
@@
 			)
 		)
-		(property "MPN" "W25Q64JVXGIM"
+		(property "MPN" "BY25Q64ESCIG(R)"
 			(at 100.33 231.775 0)
 			(effects
@@
 			)
 		)
-		(property "JLC" "C5440778"
+		(property "JLC" "C50176394"
 			(at 48.26 229.235 0)
 			(effects
@@
 			)
 		)
-		(property "LCSC" "C5440778"
+		(property "LCSC" "C50176394"
 			(at 48.26 229.235 0)
 			(effects
@@
 			)
 		)
-		(property "Manufacturer" "Winbond"
+		(property "Manufacturer" "BOYAMICRO"
 			(at 48.26 229.235 0)
 			(effects

Commit message: flash: author the LGA-8 footprint into poly_kb.pretty instead of the stock library
The Footprint field pointed at Package_SON:SON-8-1EP_3x2mm_P0.5mm_EP1.4x1.6mm,
but Package_SON is not in the project fp-lib-table - all 11 entries there are
project-local or ThirdParty - so it resolved only through KiCad's global table
and broke the repo's self-contained pattern. Now a local footprint, built from
the Boya datasheet Rev 2.6 section 9.5 rather than by analogy.

Geometry from the section 9.5 nominals: D 2.00, E 3.00, pitch 0.50 BSC, span
Nd 1.50 BSC, pad b 0.25 x L 0.45. Signal lands are 0.25 x 0.60 - the extra
0.15mm is an outward toe, since LGA has no side-wettable flank and without it
there is no inspectable fillet. Adjacent lands keep a 0.25mm gap.

Two things read off the drawing rather than assumed. Pin order follows the 9.5
Top View - 4,3,2,1 left to right along the top edge, 5,6,7,8 along the bottom -
which is rotated 90 degrees from the superseded DFN_XGIQ TR_WIN, worth knowing
before the layout pass. And pad 9 is the exposed pad, which Note 1 states is
floating inside the package; its height is not unambiguously dimensioned, so
the land is deliberately undersized at 1.50 x 1.00, clearing the signal lands
by 0.55mm. Tying it to GND is harmless as there is no internal connection, and
the board already has that net on pad 9.

Also corrects the LED footprint's descr. It claimed the pin numbers came from
'the datasheet function table', but the XL-3332RGBC datasheet does not number
its pins at all - it labels them by name only. The numbering comes from the
KiCad LED:WS2812B symbol (1 VDD, 2 DOUT, 3 VSS, 4 DIN), corroborated by the
nets on the working v3.2 boards; the sibling XL-3030RGBC datasheet does carry a
numbered table and agrees.

Co-Authored-By: Claude Opus 5 <noreply@anthropic.com>
Claude-Session: https://claude.ai/code/session_013TdVkG4xm84QHBhBEYQUBe
Parts:
- U9: footprint Package_SON:SON-8-1EP_3x2mm_P0.5mm_EP1.4x1.6mm -> poly_kb:BY25Q64ES-LGA8-2x3
Changed lines of the file:
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@@
 			)
 		)
-		(property "Footprint" "Package_SON:SON-8-1EP_3x2mm_P0.5mm_EP1.4x1.6mm"
+		(property "Footprint" "poly_kb:BY25Q64ES-LGA8-2x3"
 			(at 100.33 226.695 0)
 			(effects

Commit message: USB-C: bring HRO-TYPE-C-31-M-12-Assembly into poly_kb.pretty, repoint the schematics
The EnvUSB library (thirdparty/EnvOpenPico/.../HRO-TYPE-C31-M-12.pretty) is not
in this repo, so KiCad reports it missing on open. It was the only one of the
eight missing footprint libraries genuinely in use - the other seven are dead
references, and Nexperia595 turned out to be vestigial too, appearing only in a
lib_symbols cache while all nine 74HC595 instances already use poly_kb.

Nothing was broken, because the footprint is embedded in all four boards, but
Update PCB from Schematic could not resolve it - which is exactly what the
coming layout pass needs. Since it was embedded, it could be recovered from the
tree rather than hunted upstream: extracted from poly_kybd_split72_left USB1 and
stripped of instance-only data (42 uuids, 1 sheet path, 16 pad nets, the
placement, the USB1 reference).

Validated rather than assumed: parens balanced 300/300, 14 distinct pad names
with geometry identical to the board, 13 graphic elements kept, and the board
instance carried no descr or 3D model, so nothing was lost.

Kept on B.Cu deliberately. All eight instances across the four boards are
bottom-mounted, so there is no front-side instance to copy, and keeping the
as-built side avoids a front/back mirroring transformation that has no
reference to verify against - the failure mode there is a silently mirrored
connector. The provenance and this reasoning are recorded in the footprint's
descr.

Schematics: 5 instances repointed from EnvUSB: to poly_kb: - USB1 in
rp_pico.kicad_sch and USB2 in both split72 and both split42 top sheets. No
lib_symbols cache carried the reference, so none had to be touched.

The boards still name EnvUSB: for the placed footprints. That is inert - the
geometry is embedded and identical - and the next Update PCB from Schematic
will swap them to the poly_kb name.

Co-Authored-By: Claude Opus 5 <noreply@anthropic.com>
Claude-Session: https://claude.ai/code/session_013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
Parts:
- USB1: footprint EnvUSB:HRO-TYPE-C-31-M-12-Assembly -> poly_kb:HRO-TYPE-C-31-M-12-Assembly
Changed lines of the file:
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@@
 			)
 		)
-		(property "Footprint" "EnvUSB:HRO-TYPE-C-31-M-12-Assembly"
+		(property "Footprint" "poly_kb:HRO-TYPE-C-31-M-12-Assembly"
 			(at 36.83 95.25 0)
 			(effects
