File: poly_kybd/rp_pico.kicad_sch (KiCad schematic)
At the start: 46 parts, among them SW2 EVQPUC02K, SW3 EVQPUC02K, U1 TLV62569DBVR, U10 RP2040, U11 TPD4E05U06DQAR, U9 BY25Q64ESCIG(R), Y1 7M12000044

Commit message: Updated pcb layout with bigger LED footprint and smaller footprint for flash
Connections:
- net GND: no longer U9.9 (EP)
- no-connect marks 2 -> 3
Changed lines of the file:
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@@
+	)
+	(no_connect
+		(at 76.2 249.555)
 	)
 	(no_connect
@@
 		)
 	)
-	(hierarchical_label "GND"
-		(shape input)
-		(at 76.2 249.555 270)
-		(effects
-			(font
-				(size 1.27 1.27)
-			)
-			(justify right)
-		)
-	)
