File: poly_kybd/shift_registers.kicad_sch (KiCad schematic)
At the start: 5 parts, among them U4 74HC595BQ, U5 74HC595BQ, U6 74HC595BQ, U7 74HC595BQ, U8 74HC595BQ

Commit message: Revision D caps and schematics part cleanup
Parts:
- U4, U5, U6, U7, U8: JLC (none) -> C3303719; LCSC (none) -> C3303719
Changed lines of the file:
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@@
+      (effects (font (size 1.27 1.27)) hide)
+    )
+    (property "JLC" "C3303719" (at 203.2 90.17 0)
+      (effects (font (size 1.27 1.27)) hide)
+    )
+    (property "LCSC" "C3303719" (at 203.2 90.17 0)
       (effects (font (size 1.27 1.27)) hide)
     )
@@
       (effects (font (size 1.27 1.27)) hide)
     )
+    (property "JLC" "C3303719" (at 52.07 90.17 0)
+      (effects (font (size 1.27 1.27)) hide)
+    )
+    (property "LCSC" "C3303719" (at 52.07 90.17 0)
+      (effects (font (size 1.27 1.27)) hide)
+    )
     (pin "1")
     (pin "10")
@@
       (effects (font (size 1.27 1.27)) hide)
     )
+    (property "JLC" "C3303719" (at 255.27 90.17 0)
+      (effects (font (size 1.27 1.27)) hide)
+    )
+    (property "LCSC" "C3303719" (at 255.27 90.17 0)
+      (effects (font (size 1.27 1.27)) hide)
+    )
     (pin "1")
     (pin "10")
@@
       (effects (font (size 1.27 1.27)) hide)
     )
+    (property "JLC" "C3303719" (at 160.02 90.17 0)
+      (effects (font (size 1.27 1.27)) hide)
+    )
+    (property "LCSC" "C3303719" (at 160.02 90.17 0)
+      (effects (font (size 1.27 1.27)) hide)
+    )
     (pin "1")
     (pin "10")
@@
       (effects (font (size 1.27 1.27)) hide)
     )
+    (property "JLC" "C3303719" (at 104.14 90.17 0)
+      (effects (font (size 1.27 1.27)) hide)
+    )
+    (property "LCSC" "C3303719" (at 104.14 90.17 0)
+      (effects (font (size 1.27 1.27)) hide)
+    )

Commit message: Updated left side for RoHS
Parts:
- U4, U5, U6, U7, U8: Manufacturer (none) -> Nexperia; RoHS (none) -> x
Other:
- title: (none) -> Shift Registers
Changed lines of the file:
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@@
   (paper "A4")
   (title_block
-    (date "2023-03-09")
+    (title "Shift Registers")
+    (date "2024-10-11")
+    (rev "3.2")
   )
   (wire (pts (xy 130.81 80.01) (xy 130.81 100.33))
@@
     )
     (property "LCSC" "C3303719" (at 203.2 90.17 0)
+      (effects (font (size 1.27 1.27)) hide)
+    )
+    (property "Manufacturer" "Nexperia" (at 203.2 90.17 0)
+      (effects (font (size 1.27 1.27)) hide)
+    )
+    (property "RoHS" "x" (at 203.2 90.17 0)
       (effects (font (size 1.27 1.27)) hide)
     )
@@
       (effects (font (size 1.27 1.27)) hide)
     )
+    (property "Manufacturer" "Nexperia" (at 52.07 90.17 0)
+      (effects (font (size 1.27 1.27)) hide)
+    )
+    (property "RoHS" "x" (at 52.07 90.17 0)
+      (effects (font (size 1.27 1.27)) hide)
+    )
     (pin "1")
     (pin "10")
@@
       (effects (font (size 1.27 1.27)) hide)
     )
+    (property "Manufacturer" "Nexperia" (at 255.27 90.17 0)
+      (effects (font (size 1.27 1.27)) hide)
+    )
+    (property "RoHS" "x" (at 255.27 90.17 0)
+      (effects (font (size 1.27 1.27)) hide)
+    )
     (pin "1")
     (pin "10")
@@
       (effects (font (size 1.27 1.27)) hide)
     )
+    (property "Manufacturer" "Nexperia" (at 160.02 90.17 0)
+      (effects (font (size 1.27 1.27)) hide)
+    )
+    (property "RoHS" "x" (at 160.02 90.17 0)
+      (effects (font (size 1.27 1.27)) hide)
+    )
     (pin "1")
     (pin "10")
@@
       (effects (font (size 1.27 1.27)) hide)
     )
+    (property "Manufacturer" "Nexperia" (at 104.14 90.17 0)
+      (effects (font (size 1.27 1.27)) hide)
+    )
+    (property "RoHS" "x" (at 104.14 90.17 0)
+      (effects (font (size 1.27 1.27)) hide)
+    )
