File: poly_kybd/variations/poly_corne/poly_corne_split42_right.kicad_sch (KiCad schematic)
At the start: 48 parts, among them J37 FH34SRJ-12S-0.5SH, J38 Conn_01x05, J39 FH12-30S-0.5SH, SW1 RotaryEncoder_Switch, U2 TLV62569DBVR, U26 TPD4E05U06DQAR, U3 SY6280AAC

Commit message: A5: replace four EOL parts across schematics, PCBs and the project library
All four were discontinued at JLCPCB ("no longer manufactured", 0 stock),
so the v3.2 BOM can no longer be ordered as-is. Metadata only - every
replacement keeps the same footprint, so no layout or netlist changes.

  C118249  Sunlord  TC212A475K025Y  -> C5380411 Vishay  293D475X9025A2TE3
  C170128  Samsung  CL10C6R8DB8NNNC -> C318672  Samsung CL10C6R8CB8NNNC
  C3303719 Nexperia 74HC595BQ115    -> C730243  Nexperia 74HC595BQ,115
  C2940195 Winbond  W25Q64JVXGIQ    -> C5440778 Winbond W25Q64JVXGIM

Net cost at a 200-keyboard batch: -$4.15/keyboard, -$829/batch. The flash
carries it (-$4.76/kbd); the tantalum is the only real increase
(+$0.68/kbd, and it was the only 4.7uF/25V CASE-A with volume).

Also fixed along the way:

- MPN held the LCSC code rather than a manufacturer part number on all
  four, the same defect as the buffer in #24. Now the real MPN.
- The 74HC595 datasheet pointed at a rocelec.widen.net mirror that is now
  404. Repointed to Nexperia's own copy, verified to be the
  74HC595/74HCT595 data sheet. That URL was in poly_kb.kicad_sym too, so
  the project library and its cached copies are updated together.
- Manufacturer "winbond" -> "Winbond", "Sunlord" -> "Vishay".

Scope: the corne split42 variant shares these parts and is included -
leaving EOL codes anywhere is a trap. Library and footprint identifiers
containing "XGIQ" (lib_id, sym-lib-table path, footprint name, search
tags) are deliberately unchanged: they are names, not part numbers, and
renaming them would break the library binding.

Verified: 422 property edits across 14 files, insertions and deletions
exactly balanced, and every changed line is a (property ...) line - no
pads, nets, placements or reference designators touched.

Co-Authored-By: Claude Opus 5 <noreply@anthropic.com>
Parts:
- C11: JLC C170128 -> C318672; LCSC C170128 -> C318672; MPN C170128 -> CL10C6R8CB8NNNC
- C33, C34: JLC C118249 -> C5380411; LCSC C118249 -> C5380411; MPN C118249 -> 293D475X9025A2TE3; Manufacturer Sunlord -> Vishay
Changed lines of the file:
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@@
 			)
 		)
-		(property "Datasheet" "https://www.lcsc.com/datasheet/lcsc_datasheet_2304140030_YAGEO-RC0603JR-0722RL_C108405.pdf"
+		(property "Datasheet" "https://wmsc.lcsc.com/wmsc/upload/file/pdf/v2/lcsc/2304140030_Samsung-Electro-Mechanics-CL10C6R8CB8NNNC_C318672.pdf"
 			(at 447.04 193.04 0)
 			(effects
@@
 			)
 		)
-		(property "Datasheet" "https://www.lcsc.com/datasheet/lcsc_datasheet_2304140030_Samsung-Electro-Mechanics-CL10C6R8DB8NNNC_C170128.pdf"
+		(property "Datasheet" "https://wmsc.lcsc.com/wmsc/upload/file/pdf/v2/lcsc/2304140030_Samsung-Electro-Mechanics-CL10C6R8CB8NNNC_C318672.pdf"
 			(at 532.13 299.72 0)
 			(effects
@@
 			)
 		)
-		(property "MPN" "C170128"
+		(property "MPN" "CL10C6R8CB8NNNC"
 			(at 532.13 299.72 0)
 			(effects
@@
 			)
 		)
-		(property "JLC" "C170128"
+		(property "JLC" "C318672"
 			(at 532.13 299.72 0)
 			(effects
@@
 			)
 		)
-		(property "LCSC" "C170128"
+		(property "LCSC" "C318672"
 			(at 532.13 299.72 0)
 			(effects
@@
 			)
 		)
-		(property "Datasheet" "https://www.lcsc.com/datasheet/lcsc_datasheet_2304140030_YAGEO-AC0402FR-075K1L_C144745.pdf"
+		(property "Datasheet" "https://wmsc.lcsc.com/wmsc/upload/file/pdf/v2/lcsc/2304140030_Samsung-Electro-Mechanics-CL10C6R8CB8NNNC_C318672.pdf"
 			(at 494.03 161.29 0)
 			(effects
@@
 			)
 		)
-		(property "Datasheet" "https://www.lcsc.com/datasheet/lcsc_datasheet_2304140030_Samsung-Electro-Mechanics-CL21A106KAYNNNE_C15850.pdf"
+		(property "Datasheet" "https://www.vishay.com/docs/40002/293d.pdf"
 			(at 545.465 353.06 0)
 			(effects
@@
 			)
 		)
-		(property "Datasheet" "https://www.lcsc.com/datasheet/lcsc_datasheet_1810010229_CEC-Shenzhen-Zhenhua-XinYun-Elec-CA45-A-25V-4-7uF-K_C129569.pdf"
+		(property "Datasheet" "https://www.vishay.com/docs/40002/293d.pdf"
 			(at 447.04 306.705 0)
 			(effects
@@
 			)
 		)
-		(property "MPN" "C118249"
+		(property "MPN" "293D475X9025A2TE3"
 			(at 439.42 313.055 90)
 			(effects
@@
 			)
 		)
-		(property "JLC" "C118249"
+		(property "JLC" "C5380411"
 			(at 447.04 306.705 0)
 			(effects
@@
 			)
 		)
-		(property "LCSC" "C118249"
+		(property "LCSC" "C5380411"
 			(at 447.04 306.705 0)
 			(effects
@@
 			)
 		)
-		(property "Manufacturer" "Sunlord"
+		(property "Manufacturer" "Vishay"
 			(at 447.04 306.705 0)
 			(effects
@@
 			)
 		)
-		(property "Datasheet" "~"
+		(property "Datasheet" "https://www.vishay.com/docs/40002/293d.pdf"
 			(at 556.895 70.485 0)
 			(effects
@@
 			)
 		)
-		(property "Datasheet" "~"
+		(property "Datasheet" "https://www.vishay.com/docs/40002/293d.pdf"
 			(at 546.735 40.64 0)
 			(effects
@@
 			)
 		)
-		(property "Datasheet" "https://www.lcsc.com/datasheet/lcsc_datasheet_2304140030_Samsung-Electro-Mechanics-CL21A106KAYNNNE_C15850.pdf"
+		(property "Datasheet" "https://www.vishay.com/docs/40002/293d.pdf"
 			(at 485.14 356.87 0)
 			(effects
@@
 			)
 		)
-		(property "Datasheet" "https://www.lcsc.com/datasheet/lcsc_datasheet_1810010229_CEC-Shenzhen-Zhenhua-XinYun-Elec-CA45-A-25V-4-7uF-K_C129569.pdf"
+		(property "Datasheet" "https://www.vishay.com/docs/40002/293d.pdf"
 			(at 449.58 311.785 0)
 			(effects
@@
 			)
 		)
-		(property "MPN" "C118249"
+		(property "MPN" "293D475X9025A2TE3"
 			(at 452.755 315.595 90)
 			(effects
@@
 			)
 		)
-		(property "JLC" "C118249"
+		(property "JLC" "C5380411"
 			(at 449.58 311.785 0)
 			(effects
@@
 			)
 		)
-		(property "LCSC" "C118249"
+		(property "LCSC" "C5380411"
 			(at 449.58 311.785 0)
 			(effects
@@
 			)
 		)
-		(property "Manufacturer" "Sunlord"
+		(property "Manufacturer" "Vishay"
 			(at 449.58 311.785 0)
 			(effects
@@
 			)
 		)
-		(property "Datasheet" "~"
+		(property "Datasheet" "https://www.vishay.com/docs/40002/293d.pdf"
 			(at 541.655 70.485 0)
 			(effects
@@
 			)
 		)
-		(property "Datasheet" "https://www.lcsc.com/datasheet/lcsc_datasheet_2304140030_YAGEO-RC0603JR-0722RL_C108405.pdf"
+		(property "Datasheet" "https://www.vishay.com/docs/40002/293d.pdf"
 			(at 447.04 196.85 0)
 			(effects

Commit message: 1k 0402: retarget from Yageo C144789 to Vishay C71623
C144789 (Yageo AC0402FR-071KL) is not being restocked, and its remaining
listing carries a minimum purchase of 3,445 pieces against the 2,000
needed for a 200-keyboard batch.

Vishay CRCW04021K00FKED (C71623) is an exact functional match:

                   Yageo C144789      Vishay C71623
  value/package    1k 0402            1k 0402
  tolerance        +-1%               +-1%
  TCR              +-100ppm/C         +-100ppm/C
  power            62.5 mW            63 mW
  temperature      -55..+155 C        -55..+155 C
  stock            12,804 (min 3445)  374,486 (min 1)

Costs $0.0038 against $0.0029, so +$1.80 across a 200-keyboard batch.

R5, R6, R16, R19, R21 - 5 per board, on all four boards and in the
schematics (rp_pico.kicad_sch is shared, so its R16/R19/R21 serve every
project). 31 instances, 155 field edits.

MPN also corrected: it held the LCSC code rather than a manufacturer part
number, the same defect fixed on the buffer in #24. Datasheet repointed to
Vishay's own copy rather than an LCSC mirror.

No new RoHS evidence needed: the part carries Vishay's "e3" lead-free
termination code, and vishay-rohs-20250901.pdf - added for the tantalum -
is a company-wide statement covering all Vishay products.

Scoped strictly on JLC/LCSC == C144789, never on Manufacturer == Yageo:
212 other footprint fields on these boards are also Yageo and are
untouched. In particular AC0402FR-075K1L (the 5.1k, R3/R4/R7/R9) is a
different part in the same series and is unchanged.

Every changed line is a (property ...) line. Footprint, placement, pads
and net assignments asserted identical before and after.

Co-Authored-By: Claude Opus 5 <noreply@anthropic.com>
Parts:
- R5, R6: JLC C144789 -> C71623; LCSC C144789 -> C71623; MPN C144789 -> CRCW04021K00FKED; Manufacturer Yageo -> Vishay
Changed lines of the file:
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@@
 			)
 		)
-		(property "Datasheet" "https://www.lcsc.com/datasheet/lcsc_datasheet_2304140030_YAGEO-AC0402FR-071KL_C144789.pdf"
+		(property "Datasheet" "https://www.vishay.com/docs/20035/dcrcwe3.pdf"
 			(at 554.355 359.41 0)
 			(effects
@@
 			)
 		)
-		(property "MPN" "C144789"
+		(property "MPN" "CRCW04021K00FKED"
 			(at 554.355 359.41 0)
 			(effects
@@
 			)
 		)
-		(property "JLC" "C144789"
+		(property "JLC" "C71623"
 			(at 554.355 359.41 0)
 			(effects
@@
 			)
 		)
-		(property "LCSC" "C144789"
+		(property "LCSC" "C71623"
 			(at 554.355 359.41 0)
 			(effects
@@
 			)
 		)
-		(property "Manufacturer" "Yageo"
+		(property "Manufacturer" "Vishay"
 			(at 554.355 359.41 0)
 			(effects
@@
 			)
 		)
-		(property "Datasheet" "https://www.lcsc.com/datasheet/lcsc_datasheet_2304140030_YAGEO-AC0402FR-071KL_C144789.pdf"
+		(property "Datasheet" "https://www.vishay.com/docs/20035/dcrcwe3.pdf"
 			(at 551.18 316.23 0)
 			(effects
@@
 			)
 		)
-		(property "MPN" "C144789"
+		(property "MPN" "CRCW04021K00FKED"
 			(at 551.18 316.23 0)
 			(effects
@@
 			)
 		)
-		(property "JLC" "C144789"
+		(property "JLC" "C71623"
 			(at 551.18 316.23 0)
 			(effects
@@
 			)
 		)
-		(property "LCSC" "C144789"
+		(property "LCSC" "C71623"
 			(at 551.18 316.23 0)
 			(effects
@@
 			)
 		)
-		(property "Manufacturer" "Yageo"
+		(property "Manufacturer" "Vishay"
 			(at 551.18 316.23 0)
 			(effects

Commit message: USB-C: bring HRO-TYPE-C-31-M-12-Assembly into poly_kb.pretty, repoint the schematics
The EnvUSB library (thirdparty/EnvOpenPico/.../HRO-TYPE-C31-M-12.pretty) is not
in this repo, so KiCad reports it missing on open. It was the only one of the
eight missing footprint libraries genuinely in use - the other seven are dead
references, and Nexperia595 turned out to be vestigial too, appearing only in a
lib_symbols cache while all nine 74HC595 instances already use poly_kb.

Nothing was broken, because the footprint is embedded in all four boards, but
Update PCB from Schematic could not resolve it - which is exactly what the
coming layout pass needs. Since it was embedded, it could be recovered from the
tree rather than hunted upstream: extracted from poly_kybd_split72_left USB1 and
stripped of instance-only data (42 uuids, 1 sheet path, 16 pad nets, the
placement, the USB1 reference).

Validated rather than assumed: parens balanced 300/300, 14 distinct pad names
with geometry identical to the board, 13 graphic elements kept, and the board
instance carried no descr or 3D model, so nothing was lost.

Kept on B.Cu deliberately. All eight instances across the four boards are
bottom-mounted, so there is no front-side instance to copy, and keeping the
as-built side avoids a front/back mirroring transformation that has no
reference to verify against - the failure mode there is a silently mirrored
connector. The provenance and this reasoning are recorded in the footprint's
descr.

Schematics: 5 instances repointed from EnvUSB: to poly_kb: - USB1 in
rp_pico.kicad_sch and USB2 in both split72 and both split42 top sheets. No
lib_symbols cache carried the reference, so none had to be touched.

The boards still name EnvUSB: for the placed footprints. That is inert - the
geometry is embedded and identical - and the next Update PCB from Schematic
will swap them to the poly_kb name.

Co-Authored-By: Claude Opus 5 <noreply@anthropic.com>
Claude-Session: https://claude.ai/code/session_013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
Parts:
- USB2: footprint EnvUSB:HRO-TYPE-C-31-M-12-Assembly -> poly_kb:HRO-TYPE-C-31-M-12-Assembly
Changed lines of the file:
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@@
 			)
 		)
-		(property "Footprint" "EnvUSB:HRO-TYPE-C-31-M-12-Assembly"
+		(property "Footprint" "poly_kb:HRO-TYPE-C-31-M-12-Assembly"
 			(at 402.59 348.996 0)
 			(effects
