File: poly_kybd/variations/poly_corne/poly_corne_split42_left.kicad_pcb (KiCad board)
At the start: 4 copper layers, 134.3 x 98.5 mm, 334 parts, among them J1 FH34SRJ-14S-0.5SH, J10 FH34SRJ-14S-0.5SH, J11 FH34SRJ-14S-0.5SH, J12 FH34SRJ-14S-0.5SH, J13 FH34SRJ-14S-0.5SH, J15 FH34SRJ-14S-0.5SH, J16 FH34SRJ-14S-0.5SH, J17 FH34SRJ-14S-0.5SH, J19 FH34SRJ-14S-0.5SH, J2 FH34SRJ-14S-0.5SH, J20 FH34SRJ-14S-0.5SH, J25 FH34SRJ-14S-0.5SH, J26 FH34SRJ-14S-0.5SH, J27 FH34SRJ-14S-0.5SH, J3 FH34SRJ-14S-0.5SH, J4 FH34SRJ-14S-0.5SH, J5 FH34SRJ-14S-0.5SH, J6 FH34SRJ-14S-0.5SH, J8 FH34SRJ-14S-0.5SH, J9 FH34SRJ-14S-0.5SH, SW2 EVQPUC02K, SW3 EVQPUC02K, U1 TLV62569DBVR, U10 RP2040, U11 TPD4E05U06DQAR, U12 74AHC1G125GW,125, U13 74AHC1G125GW,125, U14 74AHC1G125GW,125, U15 74AHC1G125GW,125, U16 74AHC1G125GW,125, U17 74AHC1G125GW,125, U18 74AHC1G125GW,125, U19 74AHC1G125GW,125, U2 TLV62569DBVR, U20 74AHC1G125GW,125, U21 74AHC1G125GW,125, U22 74AHC1G125GW,125, U23 74AHC1G125GW,125, U26 TPD4E05U06DQAR, U3 SY6280AAC, U4 74HC595BQ, U5 74HC595BQ, U6 74HC595BQ, U9 W25Q64JVXGIM, Y1 7M12000044

Commit message: Keep the as-built SOT-353 land as poly_kb:SOT-353_SC-70-5_Slim
KiCad's Package_TO_SOT_SMD:SOT-353_SC-70-5 has been redrawn since these
boards were laid out: 1.025 x 0.35 roundrect at x +-0.8375, against the
as-built 0.65 x 0.40 at +-0.95. That is a 58% longer pad, and newer KiCad
flags every instance as differing from the library.

Taking the library version was measured at 189 real trace overlaps across
the four boards, hitting all 14 buffers on every board. The reason is where
the pad grows: almost all of it is at the HEEL - the inner edge moves 0.625
-> 0.325, closing the gap between the two pad columns from 1.25 mm to
0.65 mm, straight through the corridor traces use to pass under the package.
The toe gains only 0.075 mm and the pad actually gets narrower. So the
re-routing would buy heel land that sits under the body where it cannot be
inspected. Same call as the tantalum, and for the same reason.

Extracted the as-built geometry to poly_kb:SOT-353_SC-70-5_Slim - named so
it can never be mistaken for the stock footprint - and re-pointed all 54
instances plus the shared ni_buffer2.kicad_sch that drives them. Verified
per board that geometry, pad nets and placement are unchanged.

Also updated 14 stale Footprint properties on split42_right (the only board
carrying them, which would otherwise have pulled the old footprint back at
the next Update PCB from Schematic), and brought RoHS/schematics/parts.csv
in line with this month's other changes: U9 to the Boya part, C3/C8 to
Samsung, and the tantalum and RP2040 footprints to poly_kb.

Recorded in the investigate-kicad-pcb skill that the GitHub kicad-footprints
repo is stale - it still serves KiCad-5 (module ...) files over HTTP 200, and
reading it produced a confident and wrong "this footprint has not drifted".
The live library is on GitLab; the format of the header tells them apart.
Parts:
- U12, U13, U14, U15, U16, U17, U18, U19, U20, U21, U22, U23: footprint Package_TO_SOT_SMD:SOT-353_SC-70-5 -> poly_kb:SOT-353_SC-70-5_Slim
Changed lines of the file:
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@@
 		)
 	)
-	(footprint "Package_TO_SOT_SMD:SOT-353_SC-70-5"
+	(footprint "poly_kb:SOT-353_SC-70-5_Slim"
 		(layer "B.Cu")
 		(at 140.1351 46.8351)
@@
 		)
 	)
-	(footprint "Package_TO_SOT_SMD:SOT-353_SC-70-5"
+	(footprint "poly_kb:SOT-353_SC-70-5_Slim"
 		(layer "B.Cu")
 		(at 158.85 49.15)
@@
 		)
 	)
-	(footprint "Package_TO_SOT_SMD:SOT-353_SC-70-5"
+	(footprint "poly_kb:SOT-353_SC-70-5_Slim"
 		(layer "B.Cu")
 		(at 179.004 54.976)
@@
 		)
 	)
-	(footprint "Package_TO_SOT_SMD:SOT-353_SC-70-5"
+	(footprint "poly_kb:SOT-353_SC-70-5_Slim"
 		(layer "B.Cu")
 		(at 82.35 50.85)
@@
 		)
 	)
-	(footprint "Package_TO_SOT_SMD:SOT-353_SC-70-5"
+	(footprint "poly_kb:SOT-353_SC-70-5_Slim"
 		(layer "B.Cu")
 		(at 120.4 46.7)
@@
 		(embedded_fonts no)
 	)
-	(footprint "Package_TO_SOT_SMD:SOT-353_SC-70-5"
+	(footprint "poly_kb:SOT-353_SC-70-5_Slim"
 		(layer "B.Cu")
 		(at 86.4 50.55)
@@
 		)
 	)
-	(footprint "Package_TO_SOT_SMD:SOT-353_SC-70-5"
+	(footprint "poly_kb:SOT-353_SC-70-5_Slim"
 		(layer "B.Cu")
 		(at 162.55 48.35)
@@
 		)
 	)
-	(footprint "Package_TO_SOT_SMD:SOT-353_SC-70-5"
+	(footprint "poly_kb:SOT-353_SC-70-5_Slim"
 		(layer "B.Cu")
 		(at 124.5 43.7)
@@
 		)
 	)
-	(footprint "Package_TO_SOT_SMD:SOT-353_SC-70-5"
+	(footprint "poly_kb:SOT-353_SC-70-5_Slim"
 		(layer "B.Cu")
 		(at 66.36 65.42)
@@
 		)
 	)
-	(footprint "Package_TO_SOT_SMD:SOT-353_SC-70-5"
+	(footprint "poly_kb:SOT-353_SC-70-5_Slim"
 		(layer "B.Cu")
 		(at 105.5 45.9)
@@
 		)
 	)
-	(footprint "Package_TO_SOT_SMD:SOT-353_SC-70-5"
+	(footprint "poly_kb:SOT-353_SC-70-5_Slim"
 		(layer "B.Cu")
 		(at 143.5 46)
@@
 		)
 	)
-	(footprint "Package_TO_SOT_SMD:SOT-353_SC-70-5"
+	(footprint "poly_kb:SOT-353_SC-70-5_Slim"
 		(layer "B.Cu")
 		(at 101.35 50.45)
